Commit message: working

File: description/snake.robot.urdf.xacro (robot description, xacro)
@@ -2,3 +2,4 @@
 <robot xmlns:xacro="http://www.ros.org/wiki/xacro"  name="robot">
     <xacro:include filename="snake_robot_core.xacro"/>
+    <xacro:include filename="gazebo_control.xacro"/>
 </robot>

File: description/snake_robot_core.xacro (robot description, xacro)
@@ -43,4 +43,7 @@
         </xacro:inertial_box>
     </link>
+    <gazebo reference="head_link">
+        <material>Gazebo/White</material>
+    </gazebo>
     <joint name="head_1_joint" type="revolute">
         <parent link="head_link"/>
@@ -70,4 +73,7 @@
         </xacro:inertial_box>
     </link>
+    <gazebo reference="head_link">
+        <material>Gazebo/Black</material>
+    </gazebo>
     <joint name="1_2_joint" type="revolute">
         <parent link="link_1"/>
@@ -97,4 +103,7 @@
         </xacro:inertial_box>
     </link>
+    <gazebo reference="head_link">
+        <material>Gazebo/Blue</material>
+    </gazebo>
     <joint name="2_3_joint" type="revolute">
         <parent link="link_2"/>
@@ -124,4 +133,7 @@
         </xacro:inertial_box>
     </link>
+    <gazebo reference="head_link">
+        <material>Gazebo/White</material>
+    </gazebo>
     <joint name="3_4_joint" type="revolute">
         <parent link="link_3"/>
@@ -151,3 +163,6 @@
         </xacro:inertial_box>
     </link>
+    <gazebo reference="head_link">
+        <material>Gazebo/Blue</material>
+    </gazebo>
 </robot>
