Commit message: good but needs to fix gazebo_-control and yaml

File: description/gazebo_control.xacro (robot description, xacro)
@@ -19,5 +19,5 @@
     <!-- THIS PLUG IN NEED TO BE CHANGE IT IS JUST AN EXAMPLE FOR INCLUDING PLUG IN-->
     <!-- THIS PLUG IN NEED TO BE CHANGE IT IS JUST AN EXAMPLE FOR INCLUDING PLUG IN-->
-        <!-- This file demonstrates the use of some <gazebo> tags -->
+    <!-- This file demonstrates the use of some <gazebo> tags -->
     <!-- To include it add the following line -->
     <!-- <xacro:include filename="example_gazebo.xacro" /> -->
@@ -101,3 +101,2 @@
     </gazebo>
 </robot>
-</robot>

File: description/snake.robot.urdf.xacro (robot description, xacro)
@@ -2,4 +2,5 @@
 <robot xmlns:xacro="http://www.ros.org/wiki/xacro"  name="robot">
     <xacro:include filename="snake_robot_core.xacro"/>
-    <xacro:include filename="gazebo_control.xacro"/>
+<!-- <xacro:include filename="gazebo_control.xacro"/> -->
+    <xacro:include filename="materials.xacro" />
 </robot>

File: description/snake_robot_core.xacro (robot description, xacro)
@@ -2,16 +2,7 @@
 <robot xmlns:xacro="http://www.ros.org/wiki/xacro"  >
     <xacro:include filename="inertial_macros.xacro"/>
-    <material name="white">
-        <color rgba="1 1 1 1"/>
-    </material>
-    <material name="orange">
-        <color rgba="1 0.3 0.1 1"/>
-    </material>
-    <material name="blue">
-        <color rgba="0.2 0.2 1 1"/>
-    </material>
-    <material name="black">
-        <color rgba="0 0 0 1"/>
-    </material>
+    <!-- Constants for robot dimensions -->
+    <xacro:property name="PI" value="3.1415926535897931"/>
+    <!-- * * * * * * my file working fine * * * * * * * -->
     <!-- * * * BASE_LINK * * * -->
     <link name="base_link">
@@ -23,4 +14,5 @@
         <axis xyz="0 0 1"/>
     </joint>
+     <!-- TAIL LINK WHICH I HAVE CALLED FOR HEAD LINK -->
     <link name="head_link">
         <visual>
@@ -43,8 +35,10 @@
         </xacro:inertial_box>
     </link>
+    <!-- GAZEBO COLOR CONFIG -->
     <gazebo reference="head_link">
         <material>Gazebo/White</material>
     </gazebo>
-    <joint name="head_1_joint" type="revolute">
+    <!-- JOINT BETWEEN THE TAIL AND THE FIRST LINK -->
+    <joint name="link_head_1_joint" type="revolute">
         <parent link="head_link"/>
         <child link="link_1"/>
@@ -53,4 +47,5 @@
         <axis xyz="0 0 1"/>
     </joint>
+    <!-- LINK 1 -->
     <link name="link_1">
         <visual>
@@ -73,8 +68,10 @@
         </xacro:inertial_box>
     </link>
+        <!-- GAZEBO COLOR CONFIG -->
     <gazebo reference="head_link">
         <material>Gazebo/Black</material>
     </gazebo>
-    <joint name="1_2_joint" type="revolute">
+    <!-- JOINT BETWEEM LINK 1 AND 2 -->
+    <joint name="link_1_2_joint" type="revolute">
         <parent link="link_1"/>
         <child link="link_2"/>
@@ -83,4 +80,5 @@
         <axis xyz="0 0 1"/>
     </joint>
+    <!-- LINK 2 -->
     <link name="link_2">
         <visual>
@@ -103,8 +101,10 @@
         </xacro:inertial_box>
     </link>
+        <!-- GAZEBO COLOR CONFIG -->
     <gazebo reference="head_link">
         <material>Gazebo/Blue</material>
     </gazebo>
-    <joint name="2_3_joint" type="revolute">
+    <!--JOINT BETWEEN LINK 2 AND LINK 3 -->
+    <joint name="link_2_3_joint" type="revolute">
         <parent link="link_2"/>
         <child link="link_3"/>
@@ -113,4 +113,5 @@
         <axis xyz="0 0 1"/>
     </joint>
+    <!-- LINK 3 -->
     <link name="link_3">
         <visual>
@@ -133,8 +134,10 @@
         </xacro:inertial_box>
     </link>
+        <!-- GAZEBO COLOR CONFIG -->
     <gazebo reference="head_link">
         <material>Gazebo/White</material>
     </gazebo>
-    <joint name="3_4_joint" type="revolute">
+    <!-- JOINT BETWEEN LINK 3 AND LINK 4 ***NOTE THAT LINK 4 IS THE HEAD -->
+    <joint name="link_3_4_joint" type="revolute">
         <parent link="link_3"/>
         <child link="link_4"/>
@@ -143,4 +146,5 @@
         <axis xyz="0 0 1"/>
     </joint>
+    <!-- HEAD LINK -->
     <link name="link_4">
         <visual>
@@ -163,4 +167,5 @@
         </xacro:inertial_box>
     </link>
+    <!-- GAZEBO COLOR CONFIG -->
     <gazebo reference="head_link">
         <material>Gazebo/Blue</material>

Commit message: snake with camera link

File: description/gazebo_control.xacro (robot description, xacro)
@@ -6,31 +6,59 @@
     <!-- THIS PLUG IN NEED TO BE CHANGE IT IS JUST AN EXAMPLE FOR INCLUDING PLUG IN-->
     <!-- THIS PLUG IN NEED TO BE CHANGE IT IS JUST AN EXAMPLE FOR INCLUDING PLUG IN-->
-    <!-- THIS PLUGIN IMPORTED FROM URDF FILE FOR ROBOTIC ARM AND NEED TO BE
-        EDITED ACCORDING TO THE OTHER FILES NEEDED TO WORK PROPERLY-->
-    <gazebo>
-        <plugin name="gazebo_ros_joint_pose_trajectory"
-            filename="libgazebo_ros_joint_pose_trajectory.so">
-            <update_rate>2</update_rate>
-        </plugin>
+            <!-- **********************READ HERE ***********************-->
+            <!-- **********************READ HERE ***********************-->
+    <!-- my addition to orginal file -->
+    <!-- NEXT few LINE IS ADDED BY ME AND NEED TO CHECKED IF IT IS CORRECT-->
+    <!-- This plugin will publish the joint_states for the selected joints
+            (which robot_state_publisher can then use to broadcast the approprate tf). -->
+            <gazebo>
+                <plugin name="gazebo_ros_joint_state_publisher"
+                    filename="libgazebo_ros_joint_state_publisher.so">
+                    <update_rate>20</update_rate>
+                    <joint_name>slider_joint</joint_name>
+                    <joint_name>arm_joint</joint_name>
+                </plugin>
+            </gazebo>
+            <!-- This plugin will read a JointTrajectory message from the /set_joint_trajectory topic
+                    and move the machine accordingly. It's a bit clunky but it works. -->
+            <!-- You'll probably want to add damping to the joints to stop them it flopping around.
+                    e.g. <dynamics damping="10.0" friction="10.0"/> -->
+            <!-- Here's an example message to publish to test it:
+                    ros2 topic pub -1 /set_joint_trajectory trajectory_msgs/msg/JointTrajectory  '{header: {frame_id: world}, joint_names: [slider_joint, arm_joint], points: [  {positions: {0.8,0.6}} ]}' -->
+            <gazebo>
+                <plugin name="gazebo_ros_joint_pose_trajectory"
+                    filename="libgazebo_ros_joint_pose_trajectory.so">
+                    <update_rate>2</update_rate>
+                </plugin>
+            </gazebo>
+    <!-- **************************************************************************-->
+    <!-- limits-->
+    <max_joint_tourqe>200</max_joint_tourqe>
+    <max_joint_accelaration>200</max_joint_accelaration>
+    <!-- OUTPUT-->
+    <odometry_frame>odom</odometry_frame>
+    <robot_base_frame>head_link</robot_base_frame>
+    <publish_odom>true</publish_odom>
+    <publish_odom_tf>true</publish_odom_tf>
+    <publish_joint_tf></publish_joint_tf>
+    <gazebo reference="head_link">
+        <material>Gazebo/Green</material>
     </gazebo>
-            <!-- **********************READ HERE ***********************-->
-<!-- *****************THIS IS A COPY OF THE FILE example_gazebo.xacro IN THE SNAKE_WS ********** -->
-    <!-- THIS PLUG IN NEED TO BE CHANGE IT IS JUST AN EXAMPLE FOR INCLUDING PLUG IN-->
-    <!-- THIS PLUG IN NEED TO BE CHANGE IT IS JUST AN EXAMPLE FOR INCLUDING PLUG IN-->
-    <!-- THIS PLUG IN NEED TO BE CHANGE IT IS JUST AN EXAMPLE FOR INCLUDING PLUG IN-->
+    <gazebo reference="link_1">
+        <material>Gazebo/Blue</material>
+    </gazebo>
+    <gazebo reference="link_2">
+        <material>Gazebo/Orange</material>
+    </gazebo>
+    <gazebo reference="link_3">
+        <material>Gazebo/Green</material>
+    </gazebo>
+    <gazebo reference="link_4">
+        <material>Gazebo/Blue</material>
+    </gazebo>
+    <!-- ************************************************************************-->
     <!-- This file demonstrates the use of some <gazebo> tags -->
     <!-- To include it add the following line -->
     <!-- <xacro:include filename="example_gazebo.xacro" /> -->
-    <!-- Gazebo is unable to use the same <material> tags that are already in the URDF (that RViz uses). -->
-    <!-- Instead, we need to add gazebo tags for our links that refer to Gazebo materials -->
-    <gazebo reference="base_link">
-        <material>Gazebo/Green</material>
-    </gazebo>
-    <gazebo reference="slider_link">
-        <material>Gazebo/Blue</material>
-    </gazebo>
-    <gazebo reference="arm_link">
-        <material>Gazebo/Orange</material>
-    </gazebo>
     <!-- Gazebo requires the use of plugins to interact with other systems such as ROS. -->
     <!-- This plugin will publish the joint_states for the selected joints

File: description/snake_robot_core.xacro (robot description, xacro)
@@ -2,13 +2,16 @@
 <robot xmlns:xacro="http://www.ros.org/wiki/xacro"  >
     <xacro:include filename="inertial_macros.xacro"/>
+    <!-- <xacro:include filename="material.xacro"/> -->
     <!-- Constants for robot dimensions -->
     <xacro:property name="PI" value="3.1415926535897931"/>
     <!-- * * * * * * my file working fine * * * * * * * -->
     <!-- * * * BASE_LINK * * * -->
-    <link name="base_link">
-    </link>
-    <joint name="head_joint" type="fixed">
+    <link name="world"></link>
+ <!-- *********************what type of joint should we have here is it contineus -->
+ <!-- *********************what type of joint should we have here is it contineus -->
+ <!-- *********************what type of joint should we have here is it contineus -->
+    <joint name="head_joint" type="continuous">
         <origin xyz="0.0 0.0 0.00" />
-        <parent link="base_link"/>
+        <parent link="world"/>
         <child link="head_link"/>
         <axis xyz="0 0 1"/>
@@ -46,4 +49,5 @@
         <origin xyz="0.0 0.3 0.0" />
         <axis xyz="0 0 1"/>
+        <joint_properties damping="6.0" friction="6.0"/>
     </joint>
     <!-- LINK 1 -->
@@ -79,4 +83,5 @@
         <origin xyz="0.0 0.3 0.00" />
         <axis xyz="0 0 1"/>
+        <joint_properties damping="6.0" friction="6.0"/>
     </joint>
     <!-- LINK 2 -->
@@ -112,4 +117,5 @@
         <origin xyz="0.0 0.3 0.0" rpy="0 0 0"/>
         <axis xyz="0 0 1"/>
+        <joint_properties damping="6.0" friction="6.0"/>
     </joint>
     <!-- LINK 3 -->
@@ -145,4 +151,5 @@
         <origin xyz="0.0 0.3 0.0" rpy="0 0 0"/>
         <axis xyz="0 0 1"/>
+        <joint_properties damping="6.0" friction="6.0"/>
     </joint>
     <!-- HEAD LINK -->
@@ -171,3 +178,42 @@
         <material>Gazebo/Blue</material>
     </gazebo>
+    <!-- camera_joint describes where the camera is relative to the arm -->
+    <!-- - Even though the camera isn't moving relative to the arm, it will probably be helpful to have its own link/frame rather than just adding more visuals to the arm -->
+    <!-- - For this example, the camera_link origin will be at the centre of the camera's "sensor" -->
+    <joint name="camera_joint" type="fixed">
+        <origin xyz="0 0.3 0" rpy="0 0 0"/>
+        <parent link="link_4"/>
+        <child link="camera_link"/>
+    </joint>
+    <!-- camera_link describes the camera at the end of the arm -->
+    <!-- - It has multiple visual elements, which ultimately get combined together -->
+    <!-- - Even if we specify different materials, RViz will just colour them all the same as the first -->
+    <!-- - Although we could also specify multiple collision geometries, instead we just use a single box that encompasses the whole camera -->
+    <link name="camera_link">
+        <visual>
+            <origin xyz="0.00 0.03 0.05" rpy="0 0 0"/>
+            <geometry>
+                <box size="0.1 0.06 0.1" />
+            </geometry>
+            <material name="green">
+                <color rgba="0.2 1 0.2 1"/>
+            </material>
+        </visual>
+        <visual>
+            <origin xyz="0.0 0.09 0.05" rpy="1.5708 0 0"/>
+            <geometry>
+                <cylinder length="0.06" radius="0.04" />
+            </geometry>
+            <material name="blue" />
+        </visual>
+        <collision>
+            <origin xyz="0.0 0 0" rpy="0 0 0"/>
+            <geometry>
+                <box size="0.1 0.15 0.1" />
+            </geometry>
+        </collision>
+        <xacro:inertial_box mass="0.05" x="0.12" y="0.15" z="0.15">
+            <origin xyz="0.0 0.15 0.05" rpy="0.0 0.0 0.0"/>
+        </xacro:inertial_box>
+    </link>
 </robot>
