Commit message: fixed material in its own file and gazebo launching

File: description/gazebo_control.xacro (robot description, xacro)
@@ -1,36 +1,4 @@
 <?xml version="1.0"?>
-<robot xmlns:xacro="http://www.ros.org/wiki/xacro"  name="robot">
-    <!-- THIS PLUG IN NEED TO BE CHANGE IT IS JUST AN EXAMPLE FOR INCLUDING PLUG IN-->
-    <!-- THIS PLUG IN NEED TO BE CHANGE IT IS JUST AN EXAMPLE FOR INCLUDING PLUG IN-->
-    <!-- THIS PLUG IN NEED TO BE CHANGE IT IS JUST AN EXAMPLE FOR INCLUDING PLUG IN-->
-    <!-- THIS PLUG IN NEED TO BE CHANGE IT IS JUST AN EXAMPLE FOR INCLUDING PLUG IN-->
-    <!-- THIS PLUG IN NEED TO BE CHANGE IT IS JUST AN EXAMPLE FOR INCLUDING PLUG IN-->
-            <!-- **********************READ HERE ***********************-->
-            <!-- **********************READ HERE ***********************-->
-    <!-- my addition to orginal file -->
-    <!-- NEXT few LINE IS ADDED BY ME AND NEED TO CHECKED IF IT IS CORRECT-->
-    <!-- This plugin will publish the joint_states for the selected joints
-            (which robot_state_publisher can then use to broadcast the approprate tf). -->
-            <gazebo>
-                <plugin name="gazebo_ros_joint_state_publisher"
-                    filename="libgazebo_ros_joint_state_publisher.so">
-                    <update_rate>20</update_rate>
-                    <joint_name>slider_joint</joint_name>
-                    <joint_name>arm_joint</joint_name>
-                </plugin>
-            </gazebo>
-            <!-- This plugin will read a JointTrajectory message from the /set_joint_trajectory topic
-                    and move the machine accordingly. It's a bit clunky but it works. -->
-            <!-- You'll probably want to add damping to the joints to stop them it flopping around.
-                    e.g. <dynamics damping="10.0" friction="10.0"/> -->
-            <!-- Here's an example message to publish to test it:
-                    ros2 topic pub -1 /set_joint_trajectory trajectory_msgs/msg/JointTrajectory  '{header: {frame_id: world}, joint_names: [slider_joint, arm_joint], points: [  {positions: {0.8,0.6}} ]}' -->
-            <gazebo>
-                <plugin name="gazebo_ros_joint_pose_trajectory"
-                    filename="libgazebo_ros_joint_pose_trajectory.so">
-                    <update_rate>2</update_rate>
-                </plugin>
-            </gazebo>
-    <!-- **************************************************************************-->
+<robot xmlns:xacro="http://www.ros.org/wiki/xacro"  name="snake_robot">
     <!-- limits-->
     <max_joint_tourqe>200</max_joint_tourqe>
@@ -42,4 +10,5 @@
     <publish_odom_tf>true</publish_odom_tf>
     <publish_joint_tf></publish_joint_tf>
+            <!-- GAZEBO COLOR CONFIG -->
     <gazebo reference="head_link">
         <material>Gazebo/Green</material>
@@ -57,31 +26,42 @@
         <material>Gazebo/Blue</material>
     </gazebo>
-    <!-- ************************************************************************-->
-    <!-- This file demonstrates the use of some <gazebo> tags -->
-    <!-- To include it add the following line -->
-    <!-- <xacro:include filename="example_gazebo.xacro" /> -->
-    <!-- Gazebo requires the use of plugins to interact with other systems such as ROS. -->
+    <gazebo reference="camera_link">
+        <material>Gazebo/Blue</material>
+    </gazebo>
+    <!-- THIS PLUG IN NEED TO BE CHANGE IT IS JUST AN EXAMPLE FOR INCLUDING PLUG IN-->
+    <!-- THIS PLUG IN NEED TO BE CHANGE IT IS JUST AN EXAMPLE FOR INCLUDING PLUG IN-->
+    <!-- THIS PLUG IN NEED TO BE CHANGE IT IS JUST AN EXAMPLE FOR INCLUDING PLUG IN-->
+    <!-- THIS PLUG IN NEED TO BE CHANGE IT IS JUST AN EXAMPLE FOR INCLUDING PLUG IN-->
+    <!-- THIS PLUG IN NEED TO BE CHANGE IT IS JUST AN EXAMPLE FOR INCLUDING PLUG IN-->
+            <!-- **********************READ HERE ***********************-->
+            <!-- **********************READ HERE ***********************-->
+    <!-- my addition to orginal file -->
+    <!-- NEXT few LINE IS ADDED BY ME AND NEED TO CHECKED IF IT IS CORRECT-->
+    <!-- **************************************************************************-->
     <!-- This plugin will publish the joint_states for the selected joints
             (which robot_state_publisher can then use to broadcast the approprate tf). -->
-    <gazebo>
-        <plugin name="gazebo_ros_joint_state_publisher"
-            filename="libgazebo_ros_joint_state_publisher.so">
-            <update_rate>20</update_rate>
-            <joint_name>slider_joint</joint_name>
-            <joint_name>arm_joint</joint_name>
-        </plugin>
-    </gazebo>
-    <!-- This plugin will read a JointTrajectory message from the /set_joint_trajectory topic
-            and move the machine accordingly. It's a bit clunky but it works. -->
-    <!-- You'll probably want to add damping to the joints to stop them it flopping around.
-            e.g. <dynamics damping="10.0" friction="10.0"/> -->
-    <!-- Here's an example message to publish to test it:
-            ros2 topic pub -1 /set_joint_trajectory trajectory_msgs/msg/JointTrajectory  '{header: {frame_id: world}, joint_names: [slider_joint, arm_joint], points: [  {positions: {0.8,0.6}} ]}' -->
-    <gazebo>
-        <plugin name="gazebo_ros_joint_pose_trajectory"
-            filename="libgazebo_ros_joint_pose_trajectory.so">
-            <update_rate>2</update_rate>
-        </plugin>
-    </gazebo>
+            <gazebo>
+                <plugin name="gazebo_ros_joint_state_publisher"
+                    filename="libgazebo_ros_joint_state_publisher.so">
+                    <update_rate>20</update_rate>
+                    <joint_name>link_head_1_joint</joint_name>
+                    <joint_name>link_1_2_joint</joint_name>
+                    <joint_name>link_2_3_joint</joint_name>
+                    <joint_name>link_3_4_joint</joint_name>
+                </plugin>
+            </gazebo>
+            <!-- This plugin will read a JointTrajectory message from the /set_joint_trajectory topic
+                    and move the machine accordingly. It's a bit clunky but it works. -->
+            <!-- You'll probably want to add damping to the joints to stop them it flopping around.
+                    e.g. <dynamics damping="10.0" friction="10.0"/> -->
+            <!-- Here's an example message to publish to test it:
+                    ros2 topic pub -1 /set_joint_trajectory trajectory_msgs/msg/JointTrajectory  '{header: {frame_id: world}, joint_names: [slider_joint, arm_joint], points: [  {positions: {0.8,0.6}} ]}' -->
+               <gazebo>
+                <plugin name="gazebo_ros_joint_pose_trajectory"
+                    filename="libgazebo_ros_joint_pose_trajectory.so">
+                    <update_rate>2</update_rate>
+                </plugin>
+            </gazebo>
+    <!-- ************************************************************************-->
     <!-- The next section shows an example of adding a sensor, in this case a depth camera. -->
     <!-- Due to a quirk of how cameras work, an extra joint/link is required to create an
@@ -89,5 +69,5 @@
             look at https://www.ros.org/reps/rep-0103.html#suffix-frames for slightly more information. -->
     <!-- First, create the link and joint for the optical frame -->
-    <joint name="camera_optical_joint" type="fixed">
+    <!--<joint name="camera_optical_joint" type="fixed">
         <origin xyz="0 0 0" rpy="-1.571 0 -1.571" />
         <parent link="camera_link" />
@@ -95,4 +75,5 @@
     </joint>
     <link name="camera_link_optical"></link>
+-->
     <!-- Add a gazebo tag for the ORIGINAL camera_link (but in the plugin we reference the optical frame so that ROS can orient things correctly) -->
     <!-- Within the gazebo tag we have the sensor tag, and inside that there is (among other things) the camera tag with the camera parameters,
@@ -100,4 +81,5 @@
     <!-- Note that although visualise is set to true, it won't actually visualise the depth camera in gazebo. To see the preview,
             try swapping "depth" to "camera"-->
+<!--
     <gazebo reference="camera_link">
         <sensor type="depth" name="my_camera">
@@ -128,3 +110,4 @@
         </sensor>
     </gazebo>
+-->
 </robot>

File: description/snake.robot.urdf.xacro (robot description, xacro)
@@ -1,6 +1,5 @@
 <?xml version="1.0"?>
-<robot xmlns:xacro="http://www.ros.org/wiki/xacro"  name="robot">
+<robot xmlns:xacro="http://www.ros.org/wiki/xacro"  name="snake_robot">
     <xacro:include filename="snake_robot_core.xacro"/>
-<!-- <xacro:include filename="gazebo_control.xacro"/> -->
-    <xacro:include filename="materials.xacro" />
+    <xacro:include filename="gazebo_control.xacro"/>
 </robot>

File: description/snake_robot_core.xacro (robot description, xacro)
@@ -2,13 +2,15 @@
 <robot xmlns:xacro="http://www.ros.org/wiki/xacro"  >
     <xacro:include filename="inertial_macros.xacro"/>
-    <!-- <xacro:include filename="material.xacro"/> -->
+    <xacro:include filename="materials.xacro"/>
+    <xacro:include filename="gazebo_control.xacro"/>
     <!-- Constants for robot dimensions -->
     <xacro:property name="PI" value="3.1415926535897931"/>
     <!-- * * * * * * my file working fine * * * * * * * -->
     <!-- * * * BASE_LINK * * * -->
-    <link name="world"></link>
+   <!-- <link name="world"></link>-->
+ <!-- *********************what type of joint should we have here is it contineus and o we need world link at all-->
+ <!-- *********************what type of joint should we have here is it contineus and o we need world link at all-->
  <!-- *********************what type of joint should we have here is it contineus -->
- <!-- *********************what type of joint should we have here is it contineus -->
- <!-- *********************what type of joint should we have here is it contineus -->
+ <!--
     <joint name="head_joint" type="continuous">
         <origin xyz="0.0 0.0 0.00" />
@@ -17,4 +19,5 @@
         <axis xyz="0 0 1"/>
     </joint>
+-->
      <!-- TAIL LINK WHICH I HAVE CALLED FOR HEAD LINK -->
     <link name="head_link">
@@ -24,7 +27,5 @@
                 <box size="0.1 0.3 0.1"/>
             </geometry>
-            <material name="green">
-                <color rgba="0.2 1 0.2 1"/>
-            </material>
+            <material name="green"/>
         </visual>
         <collision>
@@ -38,8 +39,4 @@
         </xacro:inertial_box>
     </link>
-    <!-- GAZEBO COLOR CONFIG -->
-    <gazebo reference="head_link">
-        <material>Gazebo/White</material>
-    </gazebo>
     <!-- JOINT BETWEEN THE TAIL AND THE FIRST LINK -->
     <joint name="link_head_1_joint" type="revolute">
@@ -54,7 +51,5 @@
     <link name="link_1">
         <visual>
-            <material name="black">
-                <color rgba="0 0 0 1"/>
-            </material>
+            <material name="black"/>
             <origin xyz="0.0 0.15 0.05" rpy="0.0 0.0 0.0"/>
              <geometry>
@@ -72,8 +67,4 @@
         </xacro:inertial_box>
     </link>
-        <!-- GAZEBO COLOR CONFIG -->
-    <gazebo reference="head_link">
-        <material>Gazebo/Black</material>
-    </gazebo>
     <!-- JOINT BETWEEM LINK 1 AND 2 -->
     <joint name="link_1_2_joint" type="revolute">
@@ -88,7 +79,5 @@
     <link name="link_2">
         <visual>
-            <material name="orange">
-                <color rgba="1 0.3 0.1 1"/>
-            </material>
+            <material name="orange"/>
             <origin xyz="0.0 0.15 0.05" rpy="0.0 0.0 0.0"/>
             <geometry>
@@ -106,8 +95,4 @@
         </xacro:inertial_box>
     </link>
-        <!-- GAZEBO COLOR CONFIG -->
-    <gazebo reference="head_link">
-        <material>Gazebo/Blue</material>
-    </gazebo>
     <!--JOINT BETWEEN LINK 2 AND LINK 3 -->
     <joint name="link_2_3_joint" type="revolute">
@@ -122,7 +107,5 @@
     <link name="link_3">
         <visual>
-            <material name="black">
-                <color rgba="0 0 0 1"/>
-            </material>
+            <material name="black"/>
             <origin xyz="0.0 0.15 0.05" rpy="0.0 0.0 0.0"/>
             <geometry>
@@ -140,8 +123,4 @@
         </xacro:inertial_box>
     </link>
-        <!-- GAZEBO COLOR CONFIG -->
-    <gazebo reference="head_link">
-        <material>Gazebo/White</material>
-    </gazebo>
     <!-- JOINT BETWEEN LINK 3 AND LINK 4 ***NOTE THAT LINK 4 IS THE HEAD -->
     <joint name="link_3_4_joint" type="revolute">
@@ -156,7 +135,5 @@
     <link name="link_4">
         <visual>
-            <material name="orange">
-                <color rgba="1 0.3 0.1 1"/>
-            </material>
+            <material name="orange"/>
             <origin xyz="0.0 0.15 0.05" rpy="0.0 0.0 0.0"/>
             <geometry>
@@ -174,8 +151,4 @@
         </xacro:inertial_box>
     </link>
-    <!-- GAZEBO COLOR CONFIG -->
-    <gazebo reference="head_link">
-        <material>Gazebo/Blue</material>
-    </gazebo>
     <!-- camera_joint describes where the camera is relative to the arm -->
     <!-- - Even though the camera isn't moving relative to the arm, it will probably be helpful to have its own link/frame rather than just adding more visuals to the arm -->
@@ -196,7 +169,5 @@
                 <box size="0.1 0.06 0.1" />
             </geometry>
-            <material name="green">
-                <color rgba="0.2 1 0.2 1"/>
-            </material>
+            <material name="green"/>
         </visual>
         <visual>
