Commit message: 10 links and boxes fixed

File: description/gazebo_control.xacro (robot description, xacro)
@@ -21,11 +21,23 @@
     </gazebo>
     <gazebo reference="link_3">
+        <material>Gazebo/Blue</material>
+    </gazebo>
+    <gazebo reference="link_4">
         <material>Gazebo/Green</material>
     </gazebo>
-    <gazebo reference="link_4">
+    <gazebo reference="link_5">
         <material>Gazebo/Blue</material>
     </gazebo>
-    <gazebo reference="camera_link">
+    <gazebo reference="link_6">
+        <material>Gazebo/Orange</material>
+    </gazebo>
+    <gazebo reference="link_7">
+        <material>Gazebo/Green</material>
+    </gazebo>
+    <gazebo reference="link_8">
         <material>Gazebo/Blue</material>
+    </gazebo>
+    <gazebo reference="link_9">
+        <material>Gazebo/Orange</material>
     </gazebo>
     <!-- THIS PLUG IN NEED TO BE CHANGE IT IS JUST AN EXAMPLE FOR INCLUDING PLUG IN-->
@@ -44,9 +56,14 @@
                 <plugin name="gazebo_ros_joint_state_publisher"
                     filename="libgazebo_ros_joint_state_publisher.so">
-                    <update_rate>20</update_rate>
+                    <update_rate>50</update_rate>
                     <joint_name>link_head_1_joint</joint_name>
                     <joint_name>link_1_2_joint</joint_name>
                     <joint_name>link_2_3_joint</joint_name>
                     <joint_name>link_3_4_joint</joint_name>
+                    <joint_name>link_4_5_joint</joint_name>
+                    <joint_name>link_5_6_joint</joint_name>
+                    <joint_name>link_6_7_joint</joint_name>
+                    <joint_name>link_7_8_joint</joint_name>
+                    <joint_name>link_8_9_joint</joint_name>
                 </plugin>
             </gazebo>
@@ -56,58 +73,11 @@
                     e.g. <dynamics damping="10.0" friction="10.0"/> -->
             <!-- Here's an example message to publish to test it:
-                    ros2 topic pub -1 /set_joint_trajectory trajectory_msgs/msg/JointTrajectory  '{header: {frame_id: world}, joint_names: [slider_joint, arm_joint], points: [  {positions: {0.8,0.6}} ]}' -->
+                    ros2 topic pub -1 /set_joint_trajectory trajectory_msgs/msg/JointTrajectory  '{header: {frame_id: world}, joint_names: [head_link, link1_1], points: [  {positions: {0.8,0.6}} ]}' -->
                <gazebo>
                 <plugin name="gazebo_ros_joint_pose_trajectory"
                     filename="libgazebo_ros_joint_pose_trajectory.so">
-                    <update_rate>2</update_rate>
+                    <update_rate>50</update_rate>
                 </plugin>
             </gazebo>
     <!-- ************************************************************************-->
-    <!-- The next section shows an example of adding a sensor, in this case a depth camera. -->
-    <!-- Due to a quirk of how cameras work, an extra joint/link is required to create an
-            "optical frame" for the sensor. That isn't the focus for this tutorial, but you can
-            look at https://www.ros.org/reps/rep-0103.html#suffix-frames for slightly more information. -->
-    <!-- First, create the link and joint for the optical frame -->
-    <!--<joint name="camera_optical_joint" type="fixed">
-        <origin xyz="0 0 0" rpy="-1.571 0 -1.571" />
-        <parent link="camera_link" />
-        <child link="camera_link_optical" />
-    </joint>
-    <link name="camera_link_optical"></link>
--->
-    <!-- Add a gazebo tag for the ORIGINAL camera_link (but in the plugin we reference the optical frame so that ROS can orient things correctly) -->
-    <!-- Within the gazebo tag we have the sensor tag, and inside that there is (among other things) the camera tag with the camera parameters,
-            and the plugin tag with some extra parameters the plugin needs. -->
-    <!-- Note that although visualise is set to true, it won't actually visualise the depth camera in gazebo. To see the preview,
-            try swapping "depth" to "camera"-->
-<!--
-    <gazebo reference="camera_link">
-        <sensor type="depth" name="my_camera">
-            <update_rate>20</update_rate>
-            <visualize>true</visualize>
-            <camera name="cam">
-                <horizontal_fov>1.3962634</horizontal_fov>
-                <image>
-                    <width>640</width>
-                    <height>480</height>
-                    <format>R8B8G8</format>
-                </image>
-                <clip>
-                    <near>0.02</near>
-                    <far>300</far>
-                </clip>
-                <noise>
-                    <type>gaussian</type>
-                    <mean>0.0</mean>
-                    <stddev>0.007</stddev>
-                </noise>
-            </camera>
-            <plugin name="camera_controller" filename="libgazebo_ros_camera.so">
-                <frame_name>camera_link_optical</frame_name>
-                <min_depth>0.1</min_depth>
-                <max_depth>500</max_depth>
-            </plugin>
-        </sensor>
-    </gazebo>
--->
 </robot>

File: description/snake_robot_core.xacro (robot description, xacro)
@@ -23,18 +23,18 @@
     <link name="head_link">
         <visual>
-            <origin xyz="0.0 0.15 0.05" rpy="0.0 0.0 0.0"/>
-            <geometry>
-                <box size="0.1 0.3 0.1"/>
+            <origin xyz="0.0 0.035 0.02" rpy="0.0 0.0 0.0"/>
+            <geometry>
+                <box size="0.04 0.07 0.04"/>
             </geometry>
             <material name="green"/>
         </visual>
         <collision>
-            <origin xyz="0.0 0.15 0.05" />
-            <geometry>
-                <box size="0.1 0.3 0.1"/>
-            </geometry>
-        </collision>
-        <xacro:inertial_box mass="0.1" x="0.3" y="0.1" z="0.1">
-            <origin xyz="0.0 0.15 0.05" rpy="0.0 0.0 0.0"/>
+            <origin xyz="0.0 0.035 0.02" rpy="0.0 0.0 0.0"/>
+            <geometry>
+                <box size="0.04 0.07 0.04"/>
+            </geometry>
+        </collision>
+        <xacro:inertial_box mass="0.1" x="0.3" y="0.1" z="0.1">
+            <origin xyz="0.0 0.035 0.02" rpy="0.0 0.0 0.0"/>
         </xacro:inertial_box>
     </link>
@@ -44,5 +44,5 @@
         <child link="link_1"/>
         <limit lower="-1.5708" upper="1.5708" velocity="50.0" effort="1000.0"/>
-        <origin xyz="0.0 0.3 0.0" />
+        <origin xyz="0.0 0.1 0.0" rpy="0 0 0"/>
         <axis xyz="0 0 1"/>
         <joint_properties damping="6.0" friction="6.0"/>
@@ -52,17 +52,17 @@
         <visual>
             <material name="black"/>
-            <origin xyz="0.0 0.15 0.05" rpy="0.0 0.0 0.0"/>
+            <origin xyz="0.0 0.035 0.02" rpy="0.0 0.0 0.0"/>
              <geometry>
-                <box size="0.1 0.3 0.1"/>
-            </geometry>
-        </visual>
-        <collision>
-            <origin xyz="0.0 0.15 0.05" rpy="0.0 0.0 0.0"/>
-            <geometry>
-                <box size="0.1 0.3 0.1"/>
-            </geometry>
-        </collision>
-        <xacro:inertial_box mass="0.1" x="0.3" y="0.1" z="0.1">
-            <origin xyz="0.0 0.15 0.05" rpy="0.0 0.0 0.0"/>
+                <box size="0.04 0.07 0.04"/>
+            </geometry>
+        </visual>
+        <collision>
+            <origin xyz="0.0 0.035 0.02" rpy="0.0 0.0 0.0"/>
+            <geometry>
+                <box size="0.04 0.07 0.04"/>
+            </geometry>
+        </collision>
+        <xacro:inertial_box mass="0.1" x="0.3" y="0.1" z="0.1">
+            <origin xyz="0.0 0.035 0.02" rpy="0.0 0.0 0.0"/>
         </xacro:inertial_box>
     </link>
@@ -72,5 +72,5 @@
         <child link="link_2"/>
         <limit lower="-1.5708" upper="1.5708" velocity="50.0" effort="1000.0"/>
-        <origin xyz="0.0 0.3 0.00" />
+        <origin xyz="0.0 0.1 0.0" rpy="0 0 0"/>
         <axis xyz="0 0 1"/>
         <joint_properties damping="6.0" friction="6.0"/>
@@ -80,17 +80,17 @@
         <visual>
             <material name="orange"/>
-            <origin xyz="0.0 0.15 0.05" rpy="0.0 0.0 0.0"/>
-            <geometry>
-                <box size="0.1 0.3 0.1"/>
-            </geometry>
-        </visual>
-        <collision>
-            <origin xyz="0.0 0.15 0.05" rpy="0.0 0.0 0.0"/>
-            <geometry>
-                <box size="0.1 0.3 0.1"/>
-            </geometry>
-        </collision>
-        <xacro:inertial_box mass="0.1" x="0.3" y="0.1" z="0.1">
-            <origin xyz="0.0 0.15 0.05" rpy="0.0 0.0 0.0"/>
+            <origin xyz="0.0 0.035 0.02" rpy="0.0 0.0 0.0"/>
+            <geometry>
+                <box size="0.04 0.07 0.04"/>
+            </geometry>
+        </visual>
+        <collision>
+            <origin xyz="0.0 0.035 0.02" rpy="0.0 0.0 0.0"/>
+            <geometry>
+                <box size="0.04 0.07 0.04"/>
+            </geometry>
+        </collision>
+        <xacro:inertial_box mass="0.1" x="0.3" y="0.1" z="0.1">
+            <origin xyz="0.0 0.035 0.02" rpy="0.0 0.0 0.0"/>
         </xacro:inertial_box>
     </link>
@@ -100,5 +100,5 @@
         <child link="link_3"/>
         <limit lower="-1.5708" upper="1.5708" velocity="50.0" effort="1000.0"/>
-        <origin xyz="0.0 0.3 0.0" rpy="0 0 0"/>
+        <origin xyz="0.0 0.1 0.0" rpy="0 0 0"/>
         <axis xyz="0 0 1"/>
         <joint_properties damping="6.0" friction="6.0"/>
@@ -108,17 +108,17 @@
         <visual>
             <material name="black"/>
-            <origin xyz="0.0 0.15 0.05" rpy="0.0 0.0 0.0"/>
-            <geometry>
-                <box size="0.1 0.3 0.1"/>
-            </geometry>
-        </visual>
-        <collision>
-            <origin xyz="0.0 0.15 0.05" rpy="0.0 0.0 0.0"/>
-            <geometry>
-                <box size="0.1 0.3 0.1"/>
-            </geometry>
-        </collision>
-        <xacro:inertial_box mass="0.1" x="0.3" y="0.1" z="0.1">
-            <origin xyz="0.0 0.15 0.05" rpy="0.0 0.0 0.0"/>
+            <origin xyz="0.0 0.035 0.02" rpy="0.0 0.0 0.0"/>
+            <geometry>
+                <box size="0.04 0.07 0.04"/>
+            </geometry>
+        </visual>
+        <collision>
+            <origin xyz="0.0 0.035 0.02" rpy="0.0 0.0 0.0"/>
+            <geometry>
+                <box size="0.04 0.07 0.04"/>
+            </geometry>
+        </collision>
+        <xacro:inertial_box mass="0.1" x="0.3" y="0.1" z="0.1">
+            <origin xyz="0.0 0.035 0.02" rpy="0.0 0.0 0.0"/>
         </xacro:inertial_box>
     </link>
@@ -128,62 +128,165 @@
         <child link="link_4"/>
         <limit lower="-1.5708" upper="1.5708" velocity="50.0" effort="1000.0"/>
-        <origin xyz="0.0 0.3 0.0" rpy="0 0 0"/>
-        <axis xyz="0 0 1"/>
-        <joint_properties damping="6.0" friction="6.0"/>
-    </joint>
-    <!-- HEAD LINK -->
+        <origin xyz="0.0 0.1 0.0" rpy="0 0 0"/>
+        <axis xyz="0 0 1"/>
+        <joint_properties damping="6.0" friction="6.0"/>
+    </joint>
+    <!-- LINK 4-->
     <link name="link_4">
         <visual>
             <material name="orange"/>
-            <origin xyz="0.0 0.15 0.05" rpy="0.0 0.0 0.0"/>
-            <geometry>
-                <box size="0.1 0.3 0.1"/>
-            </geometry>
-        </visual>
-        <collision>
-            <origin xyz="0.0 0.15 0.05" rpy="0.0 0.0 0.0"/>
-            <geometry>
-                <box size="0.1 0.3 0.1"/>
-            </geometry>
-        </collision>
-        <xacro:inertial_box mass="0.1" x="0.3" y="0.1" z="0.1">
-            <origin xyz="0.0 0.15 0.05" rpy="0.0 0.0 0.0"/>
-        </xacro:inertial_box>
-    </link>
-    <!-- camera_joint describes where the camera is relative to the arm -->
-    <!-- - Even though the camera isn't moving relative to the arm, it will probably be helpful to have its own link/frame rather than just adding more visuals to the arm -->
-    <!-- - For this example, the camera_link origin will be at the centre of the camera's "sensor" -->
-    <joint name="camera_joint" type="fixed">
-        <origin xyz="0 0.3 0" rpy="0 0 0"/>
+            <origin xyz="0.0 0.035 0.02" rpy="0.0 0.0 0.0"/>
+            <geometry>
+                <box size="0.04 0.07 0.04"/>
+            </geometry>
+        </visual>
+        <collision>
+            <origin xyz="0.0 0.035 0.02" rpy="0.0 0.0 0.0"/>
+            <geometry>
+                <box size="0.04 0.07 0.04"/>
+            </geometry>
+        </collision>
+        <xacro:inertial_box mass="0.1" x="0.3" y="0.1" z="0.1">
+            <origin xyz="0.0 0.035 0.02" rpy="0.0 0.0 0.0"/>
+        </xacro:inertial_box>
+    </link>
+    <!-- JOINT BETWEEN LINK 4 AND LINK 5 ***NOTE THAT LINK 4 IS THE HEAD -->
+    <joint name="link_4_5_joint" type="revolute">
         <parent link="link_4"/>
-        <child link="camera_link"/>
-    </joint>
-    <!-- camera_link describes the camera at the end of the arm -->
-    <!-- - It has multiple visual elements, which ultimately get combined together -->
-    <!-- - Even if we specify different materials, RViz will just colour them all the same as the first -->
-    <!-- - Although we could also specify multiple collision geometries, instead we just use a single box that encompasses the whole camera -->
-    <link name="camera_link">
-        <visual>
-            <origin xyz="0.00 0.03 0.05" rpy="0 0 0"/>
-            <geometry>
-                <box size="0.1 0.06 0.1" />
-            </geometry>
-            <material name="green"/>
-        </visual>
-        <visual>
-            <origin xyz="0.0 0.09 0.05" rpy="1.5708 0 0"/>
-            <geometry>
-                <cylinder length="0.06" radius="0.04" />
-            </geometry>
-            <material name="blue" />
-        </visual>
-        <collision>
-            <origin xyz="0.0 0 0" rpy="0 0 0"/>
-            <geometry>
-                <box size="0.1 0.15 0.1" />
-            </geometry>
-        </collision>
-        <xacro:inertial_box mass="0.05" x="0.12" y="0.15" z="0.15">
-            <origin xyz="0.0 0.15 0.05" rpy="0.0 0.0 0.0"/>
+        <child link="link_5"/>
+        <limit lower="-1.5708" upper="1.5708" velocity="50.0" effort="1000.0"/>
+        <origin xyz="0.0 0.1 0.0" rpy="0 0 0"/>
+        <axis xyz="0 0 1"/>
+        <joint_properties damping="6.0" friction="6.0"/>
+    </joint>
+    <!--  LINK 5-->
+    <link name="link_5">
+        <visual>
+            <material name="orange"/>
+            <origin xyz="0.0 0.035 0.02" rpy="0.0 0.0 0.0"/>
+            <geometry>
+                <box size="0.04 0.07 0.04"/>
+            </geometry>
+        </visual>
+        <collision>
+            <origin xyz="0.0 0.035 0.02" rpy="0.0 0.0 0.0"/>
+            <geometry>
+                <box size="0.04 0.07 0.04"/>
+            </geometry>
+        </collision>
+        <xacro:inertial_box mass="0.1" x="0.3" y="0.1" z="0.1">
+            <origin xyz="0.0 0.035 0.02" rpy="0.0 0.0 0.0"/>
+        </xacro:inertial_box>
+    </link>
+    <!-- JOINT BETWEEN LINK 5 AND LINK 6 ***NOTE THAT LINK 4 IS THE HEAD -->
+    <joint name="link_5_6_joint" type="revolute">
+        <parent link="link_5"/>
+        <child link="link_6"/>
+        <limit lower="-1.5708" upper="1.5708" velocity="50.0" effort="1000.0"/>
+        <origin xyz="0.0 0.1 0.0" rpy="0 0 0"/>
+        <axis xyz="0 0 1"/>
+        <joint_properties damping="6.0" friction="6.0"/>
+    </joint>
+    <!--  LINK 6-->
+    <link name="link_6">
+        <visual>
+            <material name="orange"/>
+            <origin xyz="0.0 0.035 0.02" rpy="0.0 0.0 0.0"/>
+            <geometry>
+                <box size="0.04 0.07 0.04"/>
+            </geometry>
+        </visual>
+        <collision>
+            <origin xyz="0.0 0.035 0.02" rpy="0.0 0.0 0.0"/>
+            <geometry>
+                <box size="0.04 0.07 0.04"/>
+            </geometry>
+        </collision>
+        <xacro:inertial_box mass="0.1" x="0.3" y="0.1" z="0.1">
+            <origin xyz="0.0 0.035 0.02" rpy="0.0 0.0 0.0"/>
+        </xacro:inertial_box>
+    </link>
+    <!-- JOINT BETWEEN LINK 6 AND LINK 7 ***NOTE THAT LINK 4 IS THE HEAD -->
+    <joint name="link_6_7_joint" type="revolute">
+        <parent link="link_6"/>
+        <child link="link_7"/>
+        <limit lower="-1.5708" upper="1.5708" velocity="50.0" effort="1000.0"/>
+        <origin xyz="0.0 0.1 0.0" rpy="0 0 0"/>
+        <axis xyz="0 0 1"/>
+        <joint_properties damping="6.0" friction="6.0"/>
+    </joint>
+    <!--  LINK 7-->
+    <link name="link_7">
+        <visual>
+            <material name="orange"/>
+            <origin xyz="0.0 0.035 0.02" rpy="0.0 0.0 0.0"/>
+            <geometry>
+                <box size="0.04 0.07 0.04"/>
+            </geometry>
+        </visual>
+        <collision>
+            <origin xyz="0.0 0.035 0.02" rpy="0.0 0.0 0.0"/>
+            <geometry>
+                <box size="0.04 0.07 0.04"/>
+            </geometry>
+        </collision>
+        <xacro:inertial_box mass="0.1" x="0.3" y="0.1" z="0.1">
+            <origin xyz="0.0 0.035 0.02" rpy="0.0 0.0 0.0"/>
+        </xacro:inertial_box>
+    </link>
+    <!-- JOINT BETWEEN LINK 7 AND LINK 8 ***NOTE THAT LINK 4 IS THE HEAD -->
+    <joint name="link_7_8_joint" type="revolute">
+        <parent link="link_7"/>
+        <child link="link_8"/>
+        <limit lower="-1.5708" upper="1.5708" velocity="50.0" effort="1000.0"/>
+        <origin xyz="0.0 0.1 0.0" rpy="0 0 0"/>
+        <axis xyz="0 0 1"/>
+        <joint_properties damping="6.0" friction="6.0"/>
+    </joint>
+    <!--  LINK 8-->
+    <link name="link_8">
+        <visual>
+            <material name="orange"/>
+            <origin xyz="0.0 0.035 0.02" rpy="0.0 0.0 0.0"/>
+            <geometry>
+                <box size="0.04 0.07 0.04"/>
+            </geometry>
+        </visual>
+        <collision>
+            <origin xyz="0.0 0.035 0.02" rpy="0.0 0.0 0.0"/>
+            <geometry>
+                <box size="0.04 0.07 0.04"/>
+            </geometry>
+        </collision>
+        <xacro:inertial_box mass="0.1" x="0.3" y="0.1" z="0.1">
+            <origin xyz="0.0 0.035 0.02" rpy="0.0 0.0 0.0"/>
+        </xacro:inertial_box>
+    </link>
+    <!-- JOINT BETWEEN LINK 8 AND LINK 9 ***NOTE THAT LINK 4 IS THE HEAD -->
+    <joint name="link_8_9_joint" type="revolute">
+        <parent link="link_8"/>
+        <child link="link_9"/>
+        <limit lower="-1.5708" upper="1.5708" velocity="50.0" effort="1000.0"/>
+        <origin xyz="0.0 0.1 0.0" rpy="0 0 0"/>
+        <axis xyz="0 0 1"/>
+        <joint_properties damping="6.0" friction="6.0"/>
+    </joint>
+    <!--  LINK 9-->
+    <link name="link_9">
+        <visual>
+            <material name="orange"/>
+            <origin xyz="0.0 0.035 0.02" rpy="0.0 0.0 0.0"/>
+            <geometry>
+                <box size="0.04 0.07 0.04"/>
+            </geometry>
+        </visual>
+        <collision>
+            <origin xyz="0.0 0.035 0.02" rpy="0.0 0.0 0.0"/>
+            <geometry>
+                <box size="0.04 0.07 0.04"/>
+            </geometry>
+        </collision>
+        <xacro:inertial_box mass="0.1" x="0.3" y="0.1" z="0.1">
+            <origin xyz="0.0 0.035 0.02" rpy="0.0 0.0 0.0"/>
         </xacro:inertial_box>
     </link>
