Commit message: ss

File: description/snake_robot_core.xacro (robot description, xacro)
@@ -3,9 +3,9 @@
     <xacro:include filename="inertial_macros.xacro"/>
     <xacro:include filename="materials.xacro"/>
-   <!-- <xacro:include filename="gazebo_control.xacro"/> -->
+   <!-- <xacro:include filename="ros2_control.xacro"/> -->
    <xacro:include filename="ros2_control.xacro" />
-    <!-- Constants for robot dimensions -->
+   <!-- Constants for robot dimensions -->
     <xacro:property name="PI" value="3.1415926535897931"/>
-     <odometry_frame>odom</odometry_frame>
+    <odometry_frame>odom</odometry_frame>
     <robot_base_frame>head_link</robot_base_frame>
     <publish_odom>true</publish_odom>
@@ -16,57 +16,57 @@
     <link name="head_link">
         <visual>
-            <geometry>
-                      <box size="0.04 0.07 0.04"/>
+            <origin xyz="0.0 0.035 0.02" rpy="0.0 0.0 0.0"/>
+            <geometry>
+                <box size="0.04 0.07 0.04"/>
             </geometry>
             <material name="green"/>
-            <origin xyz="0.0 0.035 0.02" rpy="0.0 0.0 0.0"/>
-        </visual>
-        <collision>
-             <origin xyz="0.0 0.035 0.02"/>
-            <geometry>
-                    <box size="0.04 0.07 0.04"/>
-            </geometry>
-        </collision>
-        <xacro:inertial_box mass="1" x="0.04" y="0.07" z="0.04">
-              <origin xyz="0.0 0.035 0.02" rpy="0.0 0.0 0.0"/>
-        </xacro:inertial_box>
-      </link>
+        </visual>
+        <collision>
+            <origin xyz="0.0 0.035 0.02" rpy="0.0 0.0 0.0"/>
+            <geometry>
+                <box size="0.04 0.07 0.04"/>
+            </geometry>
+        </collision>
+        <xacro:inertial_box mass="0.1" x="0.3" y="0.1" z="0.1">
+            <origin xyz="0.0 0.035 0.02" rpy="0.0 0.0 0.0"/>
+        </xacro:inertial_box>
+    </link>
     <!-- JOINT BETWEEN THE TAIL AND THE FIRST LINK -->
     <joint name="link_head_1_joint" type="revolute">
         <parent link="head_link"/>
         <child link="link_1"/>
-        <limit lower="-0.7854" upper="0.7854" velocity="50.0" effort="1000.0"/>
-        <origin xyz="0.0 0.095 0.0" />
-        <axis xyz="0 0 1"/>
-        <joint_properties damping="6.0" friction="6.0"/>
-      </joint>
+        <limit lower="-1.5708" upper="1.5708" velocity="50.0" effort="1000.0"/>
+        <origin xyz="0.0 0.1 0.0" rpy="0 0 0"/>
+        <axis xyz="0 0 1"/>
+        <joint_properties damping="6.0" friction="6.0"/>
+    </joint>
     <!-- LINK 1 -->
     <link name="link_1">
         <visual>
-            <geometry>
-                    <box size="0.04 0.07 0.04"/>
-            </geometry>
-            <origin xyz="0.0 0.035 0.02" rpy="0.0 0.0 0.0"/>
-          <material name="black"/>
-        </visual>
-        <collision>
-            <origin xyz="0.0 0.035 0.02"/>
-            <geometry>
-                    <box size="0.04 0.07 0.04"/>
-            </geometry>
-        </collision>
-        <xacro:inertial_box mass="1" x="0.04" y="0.07" z="0.04">
-              <origin xyz="0.0 0.035 0.02" rpy="0.0 0.0 0.0"/>
-        </xacro:inertial_box>
-      </link>
+            <material name="black"/>
+            <origin xyz="0.0 0.035 0.02" rpy="0.0 0.0 0.0"/>
+             <geometry>
+                <box size="0.04 0.07 0.04"/>
+            </geometry>
+        </visual>
+        <collision>
+            <origin xyz="0.0 0.035 0.02" rpy="0.0 0.0 0.0"/>
+            <geometry>
+                <box size="0.04 0.07 0.04"/>
+            </geometry>
+        </collision>
+        <xacro:inertial_box mass="0.1" x="0.3" y="0.1" z="0.1">
+            <origin xyz="0.0 0.035 0.02" rpy="0.0 0.0 0.0"/>
+        </xacro:inertial_box>
+    </link>
     <!-- JOINT BETWEEM LINK 1 AND 2 -->
     <joint name="link_1_2_joint" type="revolute">
         <parent link="link_1"/>
         <child link="link_2"/>
-        <limit lower="-0.7854" upper="0.7854" velocity="50.0" effort="1000.0"/>
-        <origin xyz="0.0 0.095 0.0" />
-        <axis xyz="0 0 1"/>
-        <joint_properties damping="6.0" friction="6.0"/>
-      </joint>
+        <limit lower="-1.5708" upper="1.5708" velocity="50.0" effort="1000.0"/>
+        <origin xyz="0.0 0.1 0.0" rpy="0 0 0"/>
+        <axis xyz="0 0 1"/>
+        <joint_properties damping="6.0" friction="6.0"/>
+    </joint>
     <!-- LINK 2 -->
     <link name="link_2">
@@ -92,27 +92,27 @@
         <parent link="link_2"/>
         <child link="link_3"/>
-        <limit lower="-0.7854" upper="0.7854" velocity="50.0" effort="1000.0"/>
-        <origin xyz="0.0 0.095 0.0" />
-        <axis xyz="0 0 1"/>
-        <joint_properties damping="6.0" friction="6.0"/>
-      </joint>
+        <limit lower="-1.5708" upper="1.5708" velocity="50.0" effort="1000.0"/>
+        <origin xyz="0.0 0.1 0.0" rpy="0 0 0"/>
+        <axis xyz="0 0 1"/>
+        <joint_properties damping="6.0" friction="6.0"/>
+    </joint>
     <!-- LINK 3 -->
     <link name="link_3">
-            <visual>
-                <geometry>
-                        <box size="0.04 0.07 0.04"/>
-                </geometry>
-                <origin xyz="0.0 0.035 0.02" rpy="0.0 0.0 0.0"/>
-              <material name="black"/>
-            </visual>
-            <collision>
-                <origin xyz="0.0 0.035 0.02"/>
-                <geometry>
-                        <box size="0.04 0.07 0.04"/>
-                </geometry>
-            </collision>
-            <xacro:inertial_box mass="1" x="0.04" y="0.07" z="0.04">
-                  <origin xyz="0.0 0.035 0.02" rpy="0.0 0.0 0.0"/>
-            </xacro:inertial_box>
+        <visual>
+            <material name="black"/>
+            <origin xyz="0.0 0.035 0.02" rpy="0.0 0.0 0.0"/>
+            <geometry>
+                <box size="0.04 0.07 0.04"/>
+            </geometry>
+        </visual>
+        <collision>
+            <origin xyz="0.0 0.035 0.02" rpy="0.0 0.0 0.0"/>
+            <geometry>
+                <box size="0.04 0.07 0.04"/>
+            </geometry>
+        </collision>
+        <xacro:inertial_box mass="0.1" x="0.3" y="0.1" z="0.1">
+            <origin xyz="0.0 0.035 0.02" rpy="0.0 0.0 0.0"/>
+        </xacro:inertial_box>
     </link>
     <!-- JOINT BETWEEN LINK 3 AND LINK 4 ***NOTE THAT LINK 4 IS THE HEAD -->
@@ -120,26 +120,26 @@
         <parent link="link_3"/>
         <child link="link_4"/>
-        <limit lower="-0.7854" upper="0.7854" velocity="50.0" effort="1000.0"/>
-        <origin xyz="0.0 0.095 0.0" />
-        <axis xyz="0 0 1"/>
-        <joint_properties damping="6.0" friction="6.0"/>
-      </joint>
+        <limit lower="-1.5708" upper="1.5708" velocity="50.0" effort="1000.0"/>
+        <origin xyz="0.0 0.1 0.0" rpy="0 0 0"/>
+        <axis xyz="0 0 1"/>
+        <joint_properties damping="6.0" friction="6.0"/>
+    </joint>
     <!-- LINK 4-->
     <link name="link_4">
         <visual>
-            <geometry>
-                    <box size="0.04 0.07 0.04"/>
-            </geometry>
-            <origin xyz="0.0 0.035 0.02" rpy="0.0 0.0 0.0"/>
-          <material name="orange"/>
-        </visual>
-        <collision>
-            <origin xyz="0.0 0.035 0.02"/>
-            <geometry>
-                    <box size="0.04 0.07 0.04"/>
-            </geometry>
-        </collision>
-        <xacro:inertial_box mass="1" x="0.04" y="0.07" z="0.04">
-              <origin xyz="0.0 0.035 0.02" rpy="0.0 0.0 0.0"/>
+            <material name="orange"/>
+            <origin xyz="0.0 0.035 0.02" rpy="0.0 0.0 0.0"/>
+            <geometry>
+                <box size="0.04 0.07 0.04"/>
+            </geometry>
+        </visual>
+        <collision>
+            <origin xyz="0.0 0.035 0.02" rpy="0.0 0.0 0.0"/>
+            <geometry>
+                <box size="0.04 0.07 0.04"/>
+            </geometry>
+        </collision>
+        <xacro:inertial_box mass="0.1" x="0.3" y="0.1" z="0.1">
+            <origin xyz="0.0 0.035 0.02" rpy="0.0 0.0 0.0"/>
         </xacro:inertial_box>
     </link>
@@ -148,26 +148,26 @@
         <parent link="link_4"/>
         <child link="link_5"/>
-        <limit lower="-0.7854" upper="0.7854" velocity="50.0" effort="1000.0"/>
-        <origin xyz="0.0 0.095 0.0" />
-        <axis xyz="0 0 1"/>
-        <joint_properties damping="6.0" friction="6.0"/>
-      </joint>
+        <limit lower="-1.5708" upper="1.5708" velocity="50.0" effort="1000.0"/>
+        <origin xyz="0.0 0.1 0.0" rpy="0 0 0"/>
+        <axis xyz="0 0 1"/>
+        <joint_properties damping="6.0" friction="6.0"/>
+    </joint>
     <!--  LINK 5-->
     <link name="link_5">
         <visual>
-            <geometry>
-                    <box size="0.04 0.07 0.04"/>
-            </geometry>
-            <origin xyz="0.0 0.035 0.02" rpy="0.0 0.0 0.0"/>
-          <material name="black"/>
-        </visual>
-        <collision>
-            <origin xyz="0.0 0.035 0.02"/>
-            <geometry>
-                    <box size="0.04 0.07 0.04"/>
-            </geometry>
-        </collision>
-        <xacro:inertial_box mass="1" x="0.04" y="0.07" z="0.04">
-              <origin xyz="0.0 0.035 0.02" rpy="0.0 0.0 0.0"/>
+            <material name="orange"/>
+            <origin xyz="0.0 0.035 0.02" rpy="0.0 0.0 0.0"/>
+            <geometry>
+                <box size="0.04 0.07 0.04"/>
+            </geometry>
+        </visual>
+        <collision>
+            <origin xyz="0.0 0.035 0.02" rpy="0.0 0.0 0.0"/>
+            <geometry>
+                <box size="0.04 0.07 0.04"/>
+            </geometry>
+        </collision>
+        <xacro:inertial_box mass="0.1" x="0.3" y="0.1" z="0.1">
+            <origin xyz="0.0 0.035 0.02" rpy="0.0 0.0 0.0"/>
         </xacro:inertial_box>
     </link>
@@ -176,26 +176,26 @@
         <parent link="link_5"/>
         <child link="link_6"/>
-        <limit lower="-0.7854" upper="0.7854" velocity="50.0" effort="1000.0"/>
-        <origin xyz="0.0 0.095 0.0" />
-        <axis xyz="0 0 1"/>
-        <joint_properties damping="6.0" friction="6.0"/>
-      </joint>
+        <limit lower="-1.5708" upper="1.5708" velocity="50.0" effort="1000.0"/>
+        <origin xyz="0.0 0.1 0.0" rpy="0 0 0"/>
+        <axis xyz="0 0 1"/>
+        <joint_properties damping="6.0" friction="6.0"/>
+    </joint>
     <!--  LINK 6-->
     <link name="link_6">
         <visual>
-            <geometry>
-                    <box size="0.04 0.07 0.04"/>
-            </geometry>
-            <origin xyz="0.0 0.035 0.02" rpy="0.0 0.0 0.0"/>
-          <material name="orange"/>
-        </visual>
-        <collision>
-            <origin xyz="0.0 0.035 0.02"/>
-            <geometry>
-                    <box size="0.04 0.07 0.04"/>
-            </geometry>
-        </collision>
-        <xacro:inertial_box mass="1" x="0.04" y="0.07" z="0.04">
-              <origin xyz="0.0 0.035 0.02" rpy="0.0 0.0 0.0"/>
+            <material name="orange"/>
+            <origin xyz="0.0 0.035 0.02" rpy="0.0 0.0 0.0"/>
+            <geometry>
+                <box size="0.04 0.07 0.04"/>
+            </geometry>
+        </visual>
+        <collision>
+            <origin xyz="0.0 0.035 0.02" rpy="0.0 0.0 0.0"/>
+            <geometry>
+                <box size="0.04 0.07 0.04"/>
+            </geometry>
+        </collision>
+        <xacro:inertial_box mass="0.1" x="0.3" y="0.1" z="0.1">
+            <origin xyz="0.0 0.035 0.02" rpy="0.0 0.0 0.0"/>
         </xacro:inertial_box>
     </link>
@@ -204,26 +204,26 @@
         <parent link="link_6"/>
         <child link="link_7"/>
-        <limit lower="-0.7854" upper="0.7854" velocity="50.0" effort="1000.0"/>
-        <origin xyz="0.0 0.095 0.0" />
-        <axis xyz="0 0 1"/>
-        <joint_properties damping="6.0" friction="6.0"/>
-      </joint>
+        <limit lower="-1.5708" upper="1.5708" velocity="50.0" effort="1000.0"/>
+        <origin xyz="0.0 0.1 0.0" rpy="0 0 0"/>
+        <axis xyz="0 0 1"/>
+        <joint_properties damping="6.0" friction="6.0"/>
+    </joint>
     <!--  LINK 7-->
     <link name="link_7">
         <visual>
-            <geometry>
-                    <box size="0.04 0.07 0.04"/>
-            </geometry>
-            <origin xyz="0.0 0.035 0.02" rpy="0.0 0.0 0.0"/>
-          <material name="black"/>
-        </visual>
-        <collision>
-            <origin xyz="0.0 0.035 0.02"/>
-            <geometry>
-                    <box size="0.04 0.07 0.04"/>
-            </geometry>
-        </collision>
-        <xacro:inertial_box mass="1" x="0.04" y="0.07" z="0.04">
-              <origin xyz="0.0 0.035 0.02" rpy="0.0 0.0 0.0"/>
+            <material name="orange"/>
+            <origin xyz="0.0 0.035 0.02" rpy="0.0 0.0 0.0"/>
+            <geometry>
+                <box size="0.04 0.07 0.04"/>
+            </geometry>
+        </visual>
+        <collision>
+            <origin xyz="0.0 0.035 0.02" rpy="0.0 0.0 0.0"/>
+            <geometry>
+                <box size="0.04 0.07 0.04"/>
+            </geometry>
+        </collision>
+        <xacro:inertial_box mass="0.1" x="0.3" y="0.1" z="0.1">
+            <origin xyz="0.0 0.035 0.02" rpy="0.0 0.0 0.0"/>
         </xacro:inertial_box>
     </link>
@@ -232,26 +232,26 @@
         <parent link="link_7"/>
         <child link="link_8"/>
-        <limit lower="-0.7854" upper="0.7854" velocity="50.0" effort="1000.0"/>
-        <origin xyz="0.0 0.095 0.0" />
-        <axis xyz="0 0 1"/>
-        <joint_properties damping="6.0" friction="6.0"/>
-      </joint>
+        <limit lower="-1.5708" upper="1.5708" velocity="50.0" effort="1000.0"/>
+        <origin xyz="0.0 0.1 0.0" rpy="0 0 0"/>
+        <axis xyz="0 0 1"/>
+        <joint_properties damping="6.0" friction="6.0"/>
+    </joint>
     <!--  LINK 8-->
     <link name="link_8">
         <visual>
-            <geometry>
-                    <box size="0.04 0.07 0.04"/>
-            </geometry>
-            <origin xyz="0.0 0.035 0.02" rpy="0.0 0.0 0.0"/>
-          <material name="orange"/>
-        </visual>
-        <collision>
-            <origin xyz="0.0 0.035 0.02"/>
-            <geometry>
-                    <box size="0.04 0.07 0.04"/>
-            </geometry>
-        </collision>
-        <xacro:inertial_box mass="1" x="0.04" y="0.07" z="0.04">
-              <origin xyz="0.0 0.035 0.02" rpy="0.0 0.0 0.0"/>
+            <material name="orange"/>
+            <origin xyz="0.0 0.035 0.02" rpy="0.0 0.0 0.0"/>
+            <geometry>
+                <box size="0.04 0.07 0.04"/>
+            </geometry>
+        </visual>
+        <collision>
+            <origin xyz="0.0 0.035 0.02" rpy="0.0 0.0 0.0"/>
+            <geometry>
+                <box size="0.04 0.07 0.04"/>
+            </geometry>
+        </collision>
+        <xacro:inertial_box mass="0.1" x="0.3" y="0.1" z="0.1">
+            <origin xyz="0.0 0.035 0.02" rpy="0.0 0.0 0.0"/>
         </xacro:inertial_box>
     </link>
@@ -260,26 +260,26 @@
         <parent link="link_8"/>
         <child link="link_9"/>
-        <limit lower="-0.7854" upper="0.7854" velocity="50.0" effort="1000.0"/>
-        <origin xyz="0.0 0.095 0.0" />
-        <axis xyz="0 0 1"/>
-        <joint_properties damping="6.0" friction="6.0"/>
-      </joint>
+        <limit lower="-1.5708" upper="1.5708" velocity="50.0" effort="1000.0"/>
+        <origin xyz="0.0 0.1 0.0" rpy="0 0 0"/>
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
Commit message: new

File: description/snake_robot_core.xacro (robot description, xacro)
@@ -156,5 +156,5 @@
     <link name="link_5">
         <visual>
-            <material name="orange"/>
+            <material name="black"/>
             <origin xyz="0.0 0.035 0.02" rpy="0.0 0.0 0.0"/>
             <geometry>
@@ -212,5 +212,5 @@
     <link name="link_7">
         <visual>
-            <material name="orange"/>
+            <material name="black"/>
             <origin xyz="0.0 0.035 0.02" rpy="0.0 0.0 0.0"/>
             <geometry>
@@ -268,5 +268,5 @@
     <link name="link_9">
         <visual>
-            <material name="orange"/>
+            <material name="black"/>
             <origin xyz="0.0 0.035 0.02" rpy="0.0 0.0 0.0"/>
             <geometry>

Commit message: fixed space between joints

File: description/snake_robot_core.xacro (robot description, xacro)
@@ -35,6 +35,6 @@
         <parent link="link_1"/>
         <child link="link_2"/>
-        <limit lower="-1.5708" upper="1.5708" velocity="50.0" effort="1000.0"/>
-        <origin xyz="0.0 0.17 0.0" rpy="0 0 0"/>
+        <limit lower="-0.785398163397 " upper="0.785398163397" velocity="50.0" effort="1000.0"/>
+        <origin xyz="0.0 0.175 0.0" rpy="0 0 0"/>
         <axis xyz="0 0 1"/>
         <joint_properties damping="6.0" friction="6.0"/>
@@ -63,6 +63,6 @@
         <parent link="link_2"/>
         <child link="link_3"/>
-        <limit lower="-1.5708" upper="1.5708" velocity="50.0" effort="1000.0"/>
-        <origin xyz="0.0 0.17 0.0" rpy="0 0 0"/>
+        <limit lower="-0.785398163397 " upper="0.785398163397" velocity="50.0" effort="1000.0"/>
+        <origin xyz="0.0 0.175 0.0" rpy="0 0 0"/>
         <axis xyz="0 0 1"/>
         <joint_properties damping="6.0" friction="6.0"/>
@@ -91,6 +91,6 @@
         <parent link="link_3"/>
         <child link="link_4"/>
-        <limit lower="-1.5708" upper="1.5708" velocity="50.0" effort="1000.0"/>
-        <origin xyz="0.0 0.17 0.0" rpy="0 0 0"/>
+        <limit lower="-0.785398163397 " upper="0.785398163397" velocity="50.0" effort="1000.0"/>
+        <origin xyz="0.0 0.175 0.0" rpy="0 0 0"/>
         <axis xyz="0 0 1"/>
         <joint_properties damping="6.0" friction="6.0"/>
@@ -118,6 +118,6 @@
         <parent link="link_4"/>
         <child link="link_5"/>
-        <limit lower="-1.5708" upper="1.5708" velocity="50.0" effort="1000.0"/>
-        <origin xyz="0.0 0.17 0.0" rpy="0 0 0"/>
+        <limit lower="-0.785398163397 " upper="0.785398163397" velocity="50.0" effort="1000.0"/>
+        <origin xyz="0.0 0.175 0.0" rpy="0 0 0"/>
         <axis xyz="0 0 1"/>
         <joint_properties damping="6.0" friction="6.0"/>
@@ -145,6 +145,6 @@
         <parent link="link_5"/>
         <child link="link_6"/>
-        <limit lower="-1.5708" upper="1.5708" velocity="50.0" effort="1000.0"/>
-        <origin xyz="0.0 0.17 0.0" rpy="0 0 0"/>
+        <limit lower="-0.785398163397 " upper="0.785398163397" velocity="50.0" effort="1000.0"/>
+        <origin xyz="0.0 0.175 0.0" rpy="0 0 0"/>
         <axis xyz="0 0 1"/>
         <joint_properties damping="6.0" friction="6.0"/>
@@ -173,6 +173,6 @@
         <parent link="link_6"/>
         <child link="link_7"/>
-        <limit lower="-1.5708" upper="1.5708" velocity="50.0" effort="1000.0"/>
-        <origin xyz="0.0 0.17 0.0" rpy="0 0 0"/>
+        <limit lower="-0.785398163397 " upper="0.785398163397" velocity="50.0" effort="1000.0"/>
+        <origin xyz="0.0 0.175 0.0" rpy="0 0 0"/>
         <axis xyz="0 0 1"/>
         <joint_properties damping="6.0" friction="6.0"/>
@@ -201,6 +201,6 @@
         <parent link="link_7"/>
         <child link="link_8"/>
-        <limit lower="-1.5708" upper="1.5708" velocity="50.0" effort="1000.0"/>
-        <origin xyz="0.0 0.17 0.0" rpy="0 0 0"/>
+        <limit lower="-0.785398163397 " upper="0.785398163397" velocity="50.0" effort="1000.0"/>
+        <origin xyz="0.0 0.175 0.0" rpy="0 0 0"/>
         <axis xyz="0 0 1"/>
         <joint_properties damping="6.0" friction="6.0"/>
@@ -229,6 +229,6 @@
         <parent link="link_8"/>
         <child link="link_9"/>
-        <limit lower="-1.5708" upper="1.5708" velocity="50.0" effort="1000.0"/>
-        <origin xyz="0.0 0.17 0.0" rpy="0 0 0"/>
+        <limit lower="-0.785398163397 " upper="0.785398163397" velocity="50.0" effort="1000.0"/>
+        <origin xyz="0.0 0.175 0.0" rpy="0 0 0"/>
         <axis xyz="0 0 1"/>
         <joint_properties damping="6.0" friction="6.0"/>
@@ -257,6 +257,6 @@
         <parent link="link_9"/>
         <child link="link_10"/>
-        <limit lower="-1.5708" upper="1.5708" velocity="50.0" effort="1000.0"/>
-        <origin xyz="0.0 0.17 0.0" rpy="0 0 0"/>
+        <limit lower="-0.785398163397 " upper="0.785398163397" velocity="50.0" effort="1000.0"/>
+        <origin xyz="0.0 0.175 0.0" rpy="0 0 0"/>
         <axis xyz="0 0 1"/>
         <joint_properties damping="6.0" friction="6.0"/>
