Commit message: size and name update

File: description/ros2_control.xacro (robot description, xacro)
@@ -1,32 +1,32 @@
 <?xml version="1.0"?>
 <robot xmlns:xacro="http://www.ros.org/wiki/xacro"  >
-     <gazebo reference="head_link">
+     <gazebo reference="link_1">
         <material>Gazebo/Green</material>
     </gazebo>
-    <gazebo reference="link_1">
+    <gazebo reference="link_2">
         <material>Gazebo/Blue</material>
     </gazebo>
-    <gazebo reference="link_2">
+    <gazebo reference="link_3">
         <material>Gazebo/Orange</material>
     </gazebo>
-    <gazebo reference="link_3">
+    <gazebo reference="link_4">
         <material>Gazebo/Blue</material>
     </gazebo>
-    <gazebo reference="link_4">
+    <gazebo reference="link_5">
         <material>Gazebo/Green</material>
     </gazebo>
-    <gazebo reference="link_5">
+    <gazebo reference="link_6">
         <material>Gazebo/Blue</material>
     </gazebo>
-    <gazebo reference="link_6">
+    <gazebo reference="link_7">
         <material>Gazebo/Orange</material>
     </gazebo>
-    <gazebo reference="link_7">
+    <gazebo reference="link_8">
         <material>Gazebo/Green</material>
     </gazebo>
-    <gazebo reference="link_8">
+    <gazebo reference="link_9">
         <material>Gazebo/Blue</material>
     </gazebo>
-    <gazebo reference="link_9">
+    <gazebo reference="link_10">
         <material>Gazebo/Orange</material>
     </gazebo>
@@ -36,13 +36,4 @@
     	</hardware>
 <!--  ****************************************************** * * * BELOW IS Commented * *************************************************************************************** * * * * * -->
-    <joint name="link_head_1_joint">
-        <command_interface name="effort">
-            <param name="min">0</param>
-            <param name="max">200</param>
-        </command_interface>
-        <state_interface name="position"/>
-	<state_interface name="velocity"/>
-	<state_interface name="effort"/>
-    </joint>
     <joint name="link_1_2_joint">
         <command_interface name="effort">
@@ -81,5 +72,5 @@
 	<state_interface name="effort"/>
     </joint>
-      <joint name="link_5_6_joint">
+    <joint name="link_5_6_joint">
         <command_interface name="effort">
             <param name="min">0</param>
@@ -117,4 +108,13 @@
 	<state_interface name="effort"/>
     </joint>
+      <joint name="link_9_10_joint">
+        <command_interface name="effort">
+            <param name="min">0</param>
+            <param name="max">200</param>
+        </command_interface>
+        <state_interface name="position"/>
+	<state_interface name="velocity"/>
+	<state_interface name="effort"/>
+    </joint>
     </ros2_control>
     <gazebo>
@@ -122,5 +122,4 @@
                     filename="libgazebo_ros_joint_state_publisher.so">
                     <update_rate>50</update_rate>
-                    <joint_name>link_head_1_joint</joint_name>
                     <joint_name>link_1_2_joint</joint_name>
                     <joint_name>link_2_3_joint</joint_name>
@@ -131,4 +130,5 @@
                     <joint_name>link_7_8_joint</joint_name>
                     <joint_name>link_8_9_joint</joint_name>
+                    <joint_name>link_9_10_joint</joint_name>
         </plugin>
         <plugin name="gazebo_ros2_control" filename="libgazebo_ros2_control.so">

File: description/snake_robot_core.xacro (robot description, xacro)
@@ -8,62 +8,33 @@
     <xacro:property name="PI" value="3.1415926535897931"/>
     <odometry_frame>odom</odometry_frame>
-    <robot_base_frame>head_link</robot_base_frame>
+    <robot_base_frame>link_1</robot_base_frame>
     <publish_odom>true</publish_odom>
     <publish_odom_tf>true</publish_odom_tf>
     <publish_joint_tf></publish_joint_tf>
-    <!-- * * * * * * my file working fine * * * * * * * -->
-     <!-- TAIL LINK WHICH I HAVE CALLED FOR HEAD LINK -->
-    <link name="head_link">
-        <visual>
-            <origin xyz="0.0 0.035 0.02" rpy="0.0 0.0 0.0"/>
-            <geometry>
-                <box size="0.04 0.07 0.04"/>
+    <!--LINK_1 -->
+    <link name="link_1">
+        <visual>
+            <origin xyz="0.0 0.07 0.03" rpy="0.0 0.0 0.0"/>
+            <geometry>
+                <box size="0.06 0.14 0.06"/>
             </geometry>
             <material name="green"/>
         </visual>
         <collision>
-            <origin xyz="0.0 0.035 0.02" rpy="0.0 0.0 0.0"/>
-            <geometry>
-                <box size="0.04 0.07 0.04"/>
-            </geometry>
-        </collision>
-        <xacro:inertial_box mass="0.1" x="0.3" y="0.1" z="0.1">
-            <origin xyz="0.0 0.035 0.02" rpy="0.0 0.0 0.0"/>
-        </xacro:inertial_box>
-    </link>
-    <!-- JOINT BETWEEN THE TAIL AND THE FIRST LINK -->
-    <joint name="link_head_1_joint" type="revolute">
-        <parent link="head_link"/>
-        <child link="link_1"/>
-        <limit lower="-1.5708" upper="1.5708" velocity="50.0" effort="1000.0"/>
-        <origin xyz="0.0 0.1 0.0" rpy="0 0 0"/>
-        <axis xyz="0 0 1"/>
-        <joint_properties damping="6.0" friction="6.0"/>
-    </joint>
-    <!-- LINK 1 -->
-    <link name="link_1">
-        <visual>
-            <material name="black"/>
-            <origin xyz="0.0 0.035 0.02" rpy="0.0 0.0 0.0"/>
-             <geometry>
-                <box size="0.04 0.07 0.04"/>
-            </geometry>
-        </visual>
-        <collision>
-            <origin xyz="0.0 0.035 0.02" rpy="0.0 0.0 0.0"/>
-            <geometry>
-                <box size="0.04 0.07 0.04"/>
-            </geometry>
-        </collision>
-        <xacro:inertial_box mass="0.1" x="0.3" y="0.1" z="0.1">
-            <origin xyz="0.0 0.035 0.02" rpy="0.0 0.0 0.0"/>
-        </xacro:inertial_box>
-    </link>
-    <!-- JOINT BETWEEM LINK 1 AND 2 -->
+            <origin xyz="0.0 0.07 0.03" rpy="0.0 0.0 0.0"/>
+            <geometry>
+                <box size="0.06 0.14 0.06"/>
+            </geometry>
+        </collision>
+        <xacro:inertial_box mass="1" x="0.06" y="0.14" z="0.06">
+            <origin xyz="0.0 0.07 0.03" rpy="0.0 0.0 0.0"/>
+        </xacro:inertial_box>
+    </link>
+    <!-- JOINT BETWEEN THE TAIL AND THE  LINK_2 -->
     <joint name="link_1_2_joint" type="revolute">
         <parent link="link_1"/>
         <child link="link_2"/>
         <limit lower="-1.5708" upper="1.5708" velocity="50.0" effort="1000.0"/>
-        <origin xyz="0.0 0.1 0.0" rpy="0 0 0"/>
+        <origin xyz="0.0 0.17 0.0" rpy="0 0 0"/>
         <axis xyz="0 0 1"/>
         <joint_properties damping="6.0" friction="6.0"/>
@@ -72,26 +43,26 @@
     <link name="link_2">
         <visual>
-            <material name="orange"/>
-            <origin xyz="0.0 0.035 0.02" rpy="0.0 0.0 0.0"/>
-            <geometry>
-                <box size="0.04 0.07 0.04"/>
-            </geometry>
-        </visual>
-        <collision>
-            <origin xyz="0.0 0.035 0.02" rpy="0.0 0.0 0.0"/>
-            <geometry>
-                <box size="0.04 0.07 0.04"/>
-            </geometry>
-        </collision>
-        <xacro:inertial_box mass="0.1" x="0.3" y="0.1" z="0.1">
-            <origin xyz="0.0 0.035 0.02" rpy="0.0 0.0 0.0"/>
-        </xacro:inertial_box>
-    </link>
-    <!--JOINT BETWEEN LINK 2 AND LINK 3 -->
+            <material name="black"/>
+            <origin xyz="0.0 0.07 0.03" rpy="0.0 0.0 0.0"/>
+             <geometry>
+                <box size="0.06 0.14 0.06"/>
+            </geometry>
+        </visual>
+        <collision>
+            <origin xyz="0.0 0.07 0.03" rpy="0.0 0.0 0.0"/>
+            <geometry>
+                <box size="0.06 0.14 0.06"/>
+            </geometry>
+        </collision>
+        <xacro:inertial_box mass="1" x="0.06" y="0.14" z="0.06">
+            <origin xyz="0.0 0.07 0.03" rpy="0.0 0.0 0.0"/>
+        </xacro:inertial_box>
+    </link>
+    <!-- JOINT BETWEEM LINK 2 AND 3 -->
     <joint name="link_2_3_joint" type="revolute">
         <parent link="link_2"/>
         <child link="link_3"/>
         <limit lower="-1.5708" upper="1.5708" velocity="50.0" effort="1000.0"/>
-        <origin xyz="0.0 0.1 0.0" rpy="0 0 0"/>
+        <origin xyz="0.0 0.17 0.0" rpy="0 0 0"/>
         <axis xyz="0 0 1"/>
         <joint_properties damping="6.0" friction="6.0"/>
@@ -100,82 +71,80 @@
     <link name="link_3">
         <visual>
-            <material name="black"/>
-            <origin xyz="0.0 0.035 0.02" rpy="0.0 0.0 0.0"/>
-            <geometry>
-                <box size="0.04 0.07 0.04"/>
-            </geometry>
-        </visual>
-        <collision>
-            <origin xyz="0.0 0.035 0.02" rpy="0.0 0.0 0.0"/>
-            <geometry>
-                <box size="0.04 0.07 0.04"/>
-            </geometry>
-        </collision>
-        <xacro:inertial_box mass="0.1" x="0.3" y="0.1" z="0.1">
-            <origin xyz="0.0 0.035 0.02" rpy="0.0 0.0 0.0"/>
-        </xacro:inertial_box>
-    </link>
-    <!-- JOINT BETWEEN LINK 3 AND LINK 4 ***NOTE THAT LINK 4 IS THE HEAD -->
+            <material name="orange"/>
+            <origin xyz="0.0 0.07 0.03" rpy="0.0 0.0 0.0"/>
+            <geometry>
+                <box size="0.06 0.14 0.06"/>
+            </geometry>
+        </visual>
+        <collision>
+            <origin xyz="0.0 0.07 0.03" rpy="0.0 0.0 0.0"/>
+            <geometry>
+                <box size="0.06 0.14 0.06"/>
+            </geometry>
+        </collision>
+        <xacro:inertial_box mass="1" x="0.06" y="0.14" z="0.06">
+            <origin xyz="0.0 0.07 0.03" rpy="0.0 0.0 0.0"/>
+        </xacro:inertial_box>
+    </link>
+    <!--JOINT BETWEEN LINK 3 AND LINK 4 -->
     <joint name="link_3_4_joint" type="revolute">
         <parent link="link_3"/>
         <child link="link_4"/>
         <limit lower="-1.5708" upper="1.5708" velocity="50.0" effort="1000.0"/>
-        <origin xyz="0.0 0.1 0.0" rpy="0 0 0"/>
-        <axis xyz="0 0 1"/>
-        <joint_properties damping="6.0" friction="6.0"/>
-    </joint>
-    <!-- LINK 4-->
+        <origin xyz="0.0 0.17 0.0" rpy="0 0 0"/>
+        <axis xyz="0 0 1"/>
+        <joint_properties damping="6.0" friction="6.0"/>
+    </joint>
+    <!-- LINK 4 -->
     <link name="link_4">
         <visual>
-            <material name="orange"/>
-            <origin xyz="0.0 0.035 0.02" rpy="0.0 0.0 0.0"/>
-            <geometry>
-                <box size="0.04 0.07 0.04"/>
-            </geometry>
-        </visual>
-        <collision>
-            <origin xyz="0.0 0.035 0.02" rpy="0.0 0.0 0.0"/>
-            <geometry>
-                <box size="0.04 0.07 0.04"/>
-            </geometry>
-        </collision>
-        <xacro:inertial_box mass="0.1" x="0.3" y="0.1" z="0.1">
-            <origin xyz="0.0 0.035 0.02" rpy="0.0 0.0 0.0"/>
-        </xacro:inertial_box>
-    </link>
-    <!-- JOINT BETWEEN LINK 4 AND LINK 5 ***NOTE THAT LINK 4 IS THE HEAD -->
+            <material name="black"/>
+            <origin xyz="0.0 0.07 0.03" rpy="0.0 0.0 0.0"/>
+            <geometry>
+                <box size="0.06 0.14 0.06"/>
+            </geometry>
+        </visual>
+        <collision>
+            <origin xyz="0.0 0.07 0.03" rpy="0.0 0.0 0.0"/>
+            <geometry>
+                <box size="0.06 0.14 0.06"/>
+            </geometry>
+        </collision>
+        <xacro:inertial_box mass="1" x="0.06" y="0.14" z="0.06">
+            <origin xyz="0.0 0.07 0.03" rpy="0.0 0.0 0.0"/>
+        </xacro:inertial_box>
+    </link>
     <joint name="link_4_5_joint" type="revolute">
         <parent link="link_4"/>
         <child link="link_5"/>
         <limit lower="-1.5708" upper="1.5708" velocity="50.0" effort="1000.0"/>
-        <origin xyz="0.0 0.1 0.0" rpy="0 0 0"/>
-        <axis xyz="0 0 1"/>
-        <joint_properties damping="6.0" friction="6.0"/>
-    </joint>
-    <!--  LINK 5-->
+        <origin xyz="0.0 0.17 0.0" rpy="0 0 0"/>
+        <axis xyz="0 0 1"/>
+        <joint_properties damping="6.0" friction="6.0"/>
+    </joint>
+    <!-- LINK 5-->
     <link name="link_5">
         <visual>
-            <material name="black"/>
-            <origin xyz="0.0 0.035 0.02" rpy="0.0 0.0 0.0"/>
-            <geometry>
-                <box size="0.04 0.07 0.04"/>
-            </geometry>
-        </visual>
-        <collision>
-            <origin xyz="0.0 0.035 0.02" rpy="0.0 0.0 0.0"/>
-            <geometry>
-                <box size="0.04 0.07 0.04"/>
-            </geometry>
-        </collision>
-        <xacro:inertial_box mass="0.1" x="0.3" y="0.1" z="0.1">
-            <origin xyz="0.0 0.035 0.02" rpy="0.0 0.0 0.0"/>
-        </xacro:inertial_box>
-    </link>
-    <!-- JOINT BETWEEN LINK 5 AND LINK 6 ***NOTE THAT LINK 4 IS THE HEAD -->
+            <material name="orange"/>
+            <origin xyz="0.0 0.07 0.03" rpy="0.0 0.0 0.0"/>
+            <geometry>
+                <box size="0.06 0.14 0.06"/>
+            </geometry>
+        </visual>
+        <collision>
+            <origin xyz="0.0 0.07 0.03" rpy="0.0 0.0 0.0"/>
+            <geometry>
+                <box size="0.06 0.14 0.06"/>
+            </geometry>
+        </collision>
+        <xacro:inertial_box mass="1" x="0.06" y="0.14" z="0.06">
+            <origin xyz="0.0 0.07 0.03" rpy="0.0 0.0 0.0"/>
+        </xacro:inertial_box>
+    </link>
     <joint name="link_5_6_joint" type="revolute">
         <parent link="link_5"/>
         <child link="link_6"/>
         <limit lower="-1.5708" upper="1.5708" velocity="50.0" effort="1000.0"/>
-        <origin xyz="0.0 0.1 0.0" rpy="0 0 0"/>
+        <origin xyz="0.0 0.17 0.0" rpy="0 0 0"/>
         <axis xyz="0 0 1"/>
         <joint_properties damping="6.0" friction="6.0"/>
@@ -184,26 +153,26 @@
     <link name="link_6">
         <visual>
-            <material name="orange"/>
-            <origin xyz="0.0 0.035 0.02" rpy="0.0 0.0 0.0"/>
-            <geometry>
-                <box size="0.04 0.07 0.04"/>
-            </geometry>
-        </visual>
-        <collision>
-            <origin xyz="0.0 0.035 0.02" rpy="0.0 0.0 0.0"/>
-            <geometry>
-                <box size="0.04 0.07 0.04"/>
-            </geometry>
-        </collision>
-        <xacro:inertial_box mass="0.1" x="0.3" y="0.1" z="0.1">
-            <origin xyz="0.0 0.035 0.02" rpy="0.0 0.0 0.0"/>
-        </xacro:inertial_box>
-    </link>
-    <!-- JOINT BETWEEN LINK 6 AND LINK 7 ***NOTE THAT LINK 4 IS THE HEAD -->
+            <material name="black"/>
+            <origin xyz="0.0 0.07 0.03" rpy="0.0 0.0 0.0"/>
+            <geometry>
+                <box size="0.06 0.14 0.06"/>
+            </geometry>
+        </visual>
+        <collision>
+            <origin xyz="0.0 0.07 0.03" rpy="0.0 0.0 0.0"/>
+            <geometry>
+                <box size="0.06 0.14 0.06"/>
+            </geometry>
+        </collision>
+        <xacro:inertial_box mass="1" x="0.06" y="0.14" z="0.06">
+            <origin xyz="0.0 0.07 0.03" rpy="0.0 0.0 0.0"/>
+        </xacro:inertial_box>
+    </link>
+    <!-- JOINT BETWEEN LINK 6 AND LINK 7 -->
     <joint name="link_6_7_joint" type="revolute">
         <parent link="link_6"/>
         <child link="link_7"/>
         <limit lower="-1.5708" upper="1.5708" velocity="50.0" effort="1000.0"/>
-        <origin xyz="0.0 0.1 0.0" rpy="0 0 0"/>
+        <origin xyz="0.0 0.17 0.0" rpy="0 0 0"/>
         <axis xyz="0 0 1"/>
         <joint_properties damping="6.0" friction="6.0"/>
@@ -212,26 +181,26 @@
     <link name="link_7">
         <visual>
-            <material name="black"/>
-            <origin xyz="0.0 0.035 0.02" rpy="0.0 0.0 0.0"/>
-            <geometry>
-                <box size="0.04 0.07 0.04"/>
-            </geometry>
-        </visual>
-        <collision>
-            <origin xyz="0.0 0.035 0.02" rpy="0.0 0.0 0.0"/>
-            <geometry>
-                <box size="0.04 0.07 0.04"/>
-            </geometry>
-        </collision>
-        <xacro:inertial_box mass="0.1" x="0.3" y="0.1" z="0.1">
-            <origin xyz="0.0 0.035 0.02" rpy="0.0 0.0 0.0"/>
-        </xacro:inertial_box>
-    </link>
-    <!-- JOINT BETWEEN LINK 7 AND LINK 8 ***NOTE THAT LINK 4 IS THE HEAD -->
+            <material name="orange"/>
+            <origin xyz="0.0 0.07 0.03" rpy="0.0 0.0 0.0"/>
+            <geometry>
+                <box size="0.06 0.14 0.06"/>
+            </geometry>
+        </visual>
+        <collision>
+            <origin xyz="0.0 0.07 0.03" rpy="0.0 0.0 0.0"/>
+            <geometry>
+                <box size="0.06 0.14 0.06"/>
+            </geometry>
+        </collision>
+        <xacro:inertial_box mass="1" x="0.06" y="0.14" z="0.06">
+            <origin xyz="0.0 0.07 0.03" rpy="0.0 0.0 0.0"/>
+        </xacro:inertial_box>
+    </link>
+    <!-- JOINT BETWEEN LINK 7 AND LINK 8 -->
     <joint name="link_7_8_joint" type="revolute">
         <parent link="link_7"/>
         <child link="link_8"/>
         <limit lower="-1.5708" upper="1.5708" velocity="50.0" effort="1000.0"/>
-        <origin xyz="0.0 0.1 0.0" rpy="0 0 0"/>
+        <origin xyz="0.0 0.17 0.0" rpy="0 0 0"/>
         <axis xyz="0 0 1"/>
         <joint_properties damping="6.0" friction="6.0"/>
@@ -240,26 +209,26 @@
     <link name="link_8">
         <visual>
-            <material name="orange"/>
-            <origin xyz="0.0 0.035 0.02" rpy="0.0 0.0 0.0"/>
-            <geometry>
-                <box size="0.04 0.07 0.04"/>
-            </geometry>
-        </visual>
-        <collision>
-            <origin xyz="0.0 0.035 0.02" rpy="0.0 0.0 0.0"/>
-            <geometry>
-                <box size="0.04 0.07 0.04"/>
-            </geometry>
-        </collision>
-        <xacro:inertial_box mass="0.1" x="0.3" y="0.1" z="0.1">
-            <origin xyz="0.0 0.035 0.02" rpy="0.0 0.0 0.0"/>
-        </xacro:inertial_box>
-    </link>
-    <!-- JOINT BETWEEN LINK 8 AND LINK 9 ***NOTE THAT LINK 4 IS THE HEAD -->
+            <material name="black"/>
+            <origin xyz="0.0 0.07 0.03" rpy="0.0 0.0 0.0"/>
+            <geometry>
+                <box size="0.06 0.14 0.06"/>
+            </geometry>
+        </visual>
+        <collision>
+            <origin xyz="0.0 0.07 0.03" rpy="0.0 0.0 0.0"/>
+            <geometry>
+                <box size="0.06 0.14 0.06"/>
+            </geometry>
+        </collision>
+        <xacro:inertial_box mass="1" x="0.06" y="0.14" z="0.06">
+            <origin xyz="0.0 0.07 0.03" rpy="0.0 0.0 0.0"/>
+        </xacro:inertial_box>
+    </link>
+    <!-- JOINT BETWEEN LINK 8 AND LINK 9 -->
     <joint name="link_8_9_joint" type="revolute">
         <parent link="link_8"/>
         <child link="link_9"/>
         <limit lower="-1.5708" upper="1.5708" velocity="50.0" effort="1000.0"/>
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