Commit message: moving forward

File: description/ros2_control.xacro (robot description, xacro)
@@ -3,50 +3,50 @@
      <gazebo reference="link_1">
         <material>Gazebo/Orange</material>
-        <mu1>0.01</mu1>           <!--Friction coeffeceint in the direction of motion, i.e the tangential force-->
-        <mu2>1</mu2>            <!--Friction coeffeceint in the direction perpindicular to the motion, i.e the normal force-->
+        <mu1>0.1</mu1>
+        <mu2>1</mu2>
     </gazebo>
     <gazebo reference="link_2">
         <material>Gazebo/Black</material>
-        <mu1>0.01</mu1>
+        <mu1>0.1</mu1>
         <mu2>1</mu2>
     </gazebo>
     <gazebo reference="link_3">
         <material>Gazebo/Orange</material>
-        <mu1>0.01</mu1>
+        <mu1>0.1</mu1>
         <mu2>1</mu2>
     </gazebo>
     <gazebo reference="link_4">
         <material>Gazebo/Black</material>
-        <mu1>0.01</mu1>
+        <mu1>0.1</mu1>
         <mu2>1</mu2>
     </gazebo>
     <gazebo reference="link_5">
         <material>Gazebo/Orange</material>
-        <mu1>0.01</mu1>
+        <mu1>0.1</mu1>
         <mu2>1</mu2>
     </gazebo>
     <gazebo reference="link_6">
         <material>Gazebo/Black</material>
-        <mu1>0.01</mu1>
+        <mu1>0.1</mu1>
         <mu2>1</mu2>
     </gazebo>
     <gazebo reference="link_7">
         <material>Gazebo/Orange</material>
-        <mu1>0.01</mu1>
+        <mu1>0.1</mu1>
         <mu2>1</mu2>
     </gazebo>
     <gazebo reference="link_8">
         <material>Gazebo/Black</material>
-        <mu1>0.01</mu1>
+        <mu1>0.1</mu1>
         <mu2>1</mu2>
     </gazebo>
     <gazebo reference="link_9">
         <material>Gazebo/Orange</material>
-        <mu1>0.01</mu1>
+        <mu1>0.1</mu1>
         <mu2>1</mu2>
     </gazebo>
     <gazebo reference="link_10">
         <material>Gazebo/Black</material>
-        <mu1>0.01</mu1>
+        <mu1>0.1</mu1>
         <mu2>1</mu2>
     </gazebo>

File: description/snake_robot_core.xacro (robot description, xacro)
@@ -27,5 +27,5 @@
         </collision>
         <xacro:inertial_box mass="1" x="0.06" y="0.14" z="0.06">
-            <origin xyz="0.0 0.07 0.03" rpy="0.0 0.0 0.0"/>
+            <origin xyz="0.03 0.07 0.03" rpy="0.0 0.0 0.0"/>
         </xacro:inertial_box>
     </link>
@@ -34,5 +34,5 @@
         <parent link="link_1"/>
         <child link="link_2"/>
-        <limit lower="-0.785398163397 " upper="0.785398163397" velocity="10.0" effort="200.0"/>
+        <limit lower="0.785398163397 " upper="-0.785398163397" velocity="10.0" effort="200.0"/>
         <origin xyz="0.0 0.175 0.0" rpy="0 0 0"/>
         <axis xyz="0 0 1"/>
@@ -55,5 +55,5 @@
         </collision>
         <xacro:inertial_box mass="1" x="0.06" y="0.14" z="0.06">
-            <origin xyz="0.0 0.07 0.03" rpy="0.0 0.0 0.0"/>
+            <origin xyz="0.03 0.07 0.03" rpy="0.0 0.0 0.0"/>
         </xacro:inertial_box>
     </link>
@@ -62,5 +62,5 @@
         <parent link="link_2"/>
         <child link="link_3"/>
-        <limit lower="-0.785398163397 " upper="0.785398163397" velocity="10.0" effort="200.0"/>
+        <limit lower="0.785398163397 " upper="-0.785398163397" velocity="10.0" effort="200.0"/>
         <origin xyz="0.0 0.175 0.0" rpy="0 0 0"/>
         <axis xyz="0 0 1"/>
@@ -83,5 +83,5 @@
         </collision>
         <xacro:inertial_box mass="1" x="0.06" y="0.14" z="0.06">
-            <origin xyz="0.0 0.07 0.03" rpy="0.0 0.0 0.0"/>
+            <origin xyz="0.03 0.07 0.03" rpy="0.0 0.0 0.0"/>
         </xacro:inertial_box>
     </link>
@@ -90,5 +90,5 @@
         <parent link="link_3"/>
         <child link="link_4"/>
-        <limit lower="-0.785398163397 " upper="0.785398163397" velocity="10.0" effort="200.0"/>
+        <limit lower="0.785398163397 " upper="-0.785398163397" velocity="10.0" effort="200.0"/>
         <origin xyz="0.0 0.175 0.0" rpy="0 0 0"/>
         <axis xyz="0 0 1"/>
@@ -111,5 +111,5 @@
         </collision>
         <xacro:inertial_box mass="1" x="0.06" y="0.14" z="0.06">
-            <origin xyz="0.0 0.07 0.03" rpy="0.0 0.0 0.0"/>
+            <origin xyz="0.03 0.07 0.03" rpy="0.0 0.0 0.0"/>
         </xacro:inertial_box>
     </link>
@@ -117,5 +117,5 @@
         <parent link="link_4"/>
         <child link="link_5"/>
-        <limit lower="-0.785398163397 " upper="0.785398163397" velocity="10.0" effort="200.0"/>
+        <limit lower="0.785398163397 " upper="-0.785398163397" velocity="10.0" effort="200.0"/>
         <origin xyz="0.0 0.175 0.0" rpy="0 0 0"/>
         <axis xyz="0 0 1"/>
@@ -138,5 +138,5 @@
         </collision>
         <xacro:inertial_box mass="1" x="0.06" y="0.14" z="0.06">
-            <origin xyz="0.0 0.07 0.03" rpy="0.0 0.0 0.0"/>
+            <origin xyz="0.03 0.07 0.03" rpy="0.0 0.0 0.0"/>
         </xacro:inertial_box>
     </link>
@@ -144,5 +144,5 @@
         <parent link="link_5"/>
         <child link="link_6"/>
-        <limit lower="-0.785398163397 " upper="0.785398163397" velocity="10.0" effort="200.0"/>
+        <limit lower="0.785398163397 " upper="-0.785398163397" velocity="10.0" effort="200.0"/>
         <origin xyz="0.0 0.175 0.0" rpy="0 0 0"/>
         <axis xyz="0 0 1"/>
@@ -165,5 +165,5 @@
         </collision>
         <xacro:inertial_box mass="1" x="0.06" y="0.14" z="0.06">
-            <origin xyz="0.0 0.07 0.03" rpy="0.0 0.0 0.0"/>
+            <origin xyz="0.03 0.07 0.03" rpy="0.0 0.0 0.0"/>
         </xacro:inertial_box>
     </link>
@@ -172,5 +172,5 @@
         <parent link="link_6"/>
         <child link="link_7"/>
-        <limit lower="-0.785398163397 " upper="0.785398163397" velocity="10.0" effort="200.0"/>
+        <limit lower="0.785398163397 " upper="-0.785398163397" velocity="10.0" effort="200.0"/>
         <origin xyz="0.0 0.175 0.0" rpy="0 0 0"/>
         <axis xyz="0 0 1"/>
@@ -193,5 +193,5 @@
         </collision>
         <xacro:inertial_box mass="1" x="0.06" y="0.14" z="0.06">
-            <origin xyz="0.0 0.07 0.03" rpy="0.0 0.0 0.0"/>
+            <origin xyz="0.03 0.07 0.03" rpy="0.0 0.0 0.0"/>
         </xacro:inertial_box>
     </link>
@@ -200,5 +200,5 @@
         <parent link="link_7"/>
         <child link="link_8"/>
-        <limit lower="-0.785398163397 " upper="0.785398163397" velocity="10.0" effort="200.0"/>
+        <limit lower="0.785398163397 " upper="-0.785398163397" velocity="10.0" effort="200.0"/>
         <origin xyz="0.0 0.175 0.0" rpy="0 0 0"/>
         <axis xyz="0 0 1"/>
@@ -221,5 +221,5 @@
         </collision>
         <xacro:inertial_box mass="1" x="0.06" y="0.14" z="0.06">
-            <origin xyz="0.0 0.07 0.03" rpy="0.0 0.0 0.0"/>
+            <origin xyz="0.03 0.07 0.03" rpy="0.0 0.0 0.0"/>
         </xacro:inertial_box>
     </link>
@@ -228,5 +228,5 @@
         <parent link="link_8"/>
         <child link="link_9"/>
-        <limit lower="-0.785398163397 " upper="0.785398163397" velocity="10.0" effort="200.0"/>
+        <limit lower="0.785398163397 " upper="-0.785398163397" velocity="10.0" effort="200.0"/>
         <origin xyz="0.0 0.175 0.0" rpy="0 0 0"/>
         <axis xyz="0 0 1"/>
@@ -249,5 +249,5 @@
         </collision>
         <xacro:inertial_box mass="1" x="0.06" y="0.14" z="0.06">
-            <origin xyz="0.0 0.07 0.03" rpy="0.0 0.0 0.0"/>
+            <origin xyz="0.03 0.07 0.03" rpy="0.0 0.0 0.0"/>
         </xacro:inertial_box>
     </link>
@@ -277,5 +277,5 @@
         </collision>
         <xacro:inertial_box mass="1" x="0.06" y="0.14" z="0.06">
-            <origin xyz="0.0 0.07 0.03" rpy="0.0 0.0 0.0"/>
+            <origin xyz="0.03 0.07 0.03" rpy="0.0 0.0 0.0"/>
         </xacro:inertial_box>
     </link>

Commit message: forward with little drift

File: description/ros2_control.xacro (robot description, xacro)
@@ -3,51 +3,51 @@
      <gazebo reference="link_1">
         <material>Gazebo/Orange</material>
-        <mu1>0.1</mu1>
-        <mu2>1</mu2>
+        <mu1>0.05</mu1>
+        <mu2>0.5</mu2>
     </gazebo>
     <gazebo reference="link_2">
         <material>Gazebo/Black</material>
-        <mu1>0.1</mu1>
-        <mu2>1</mu2>
+        <mu1>0.05</mu1>
+        <mu2>0.5</mu2>
     </gazebo>
     <gazebo reference="link_3">
         <material>Gazebo/Orange</material>
-        <mu1>0.1</mu1>
-        <mu2>1</mu2>
+        <mu1>0.05</mu1>
+        <mu2>0.5</mu2>
     </gazebo>
     <gazebo reference="link_4">
         <material>Gazebo/Black</material>
-        <mu1>0.1</mu1>
-        <mu2>1</mu2>
+        <mu1>0.05</mu1>
+        <mu2>0.5</mu2>
     </gazebo>
     <gazebo reference="link_5">
         <material>Gazebo/Orange</material>
-        <mu1>0.1</mu1>
-        <mu2>1</mu2>
+        <mu1>0.05</mu1>
+        <mu2>0.5</mu2>
     </gazebo>
     <gazebo reference="link_6">
         <material>Gazebo/Black</material>
-        <mu1>0.1</mu1>
-        <mu2>1</mu2>
+        <mu1>0.05</mu1>
+        <mu2>0.5</mu2>
     </gazebo>
     <gazebo reference="link_7">
         <material>Gazebo/Orange</material>
-        <mu1>0.1</mu1>
-        <mu2>1</mu2>
+        <mu1>0.05</mu1>
+        <mu2>0.5</mu2>
     </gazebo>
     <gazebo reference="link_8">
         <material>Gazebo/Black</material>
-        <mu1>0.1</mu1>
-        <mu2>1</mu2>
+        <mu1>0.05</mu1>
+        <mu2>0.5</mu2>
     </gazebo>
     <gazebo reference="link_9">
         <material>Gazebo/Orange</material>
-        <mu1>0.1</mu1>
-        <mu2>1</mu2>
+        <mu1>0.05</mu1>
+        <mu2>0.5</mu2>
     </gazebo>
     <gazebo reference="link_10">
         <material>Gazebo/Black</material>
-        <mu1>0.1</mu1>
-        <mu2>1</mu2>
+        <mu1>0.05</mu1>
+        <mu2>0.5</mu2>
     </gazebo>
     <ros2_control name="GazeboSystem" type="system">

File: description/snake_robot_core.xacro (robot description, xacro)
@@ -34,8 +34,8 @@
         <parent link="link_1"/>
         <child link="link_2"/>
-        <limit lower="0.785398163397 " upper="-0.785398163397" velocity="10.0" effort="200.0"/>
-        <origin xyz="0.0 0.175 0.0" rpy="0 0 0"/>
-        <axis xyz="0 0 1"/>
-        <joint_properties damping="6.0" friction="6.0"/>
+        <limit lower="-0.785398163397 " upper="0.785398163397" velocity="10.0" effort="200.0"/>
+        <origin xyz="0.0 0.175 0.0" rpy="0 0 0"/>
+        <axis xyz="0 0 1"/>
+        <joint_properties damping="2.0" friction="2.0"/>
     </joint>
     <!-- LINK 2 -->
@@ -62,8 +62,8 @@
         <parent link="link_2"/>
         <child link="link_3"/>
-        <limit lower="0.785398163397 " upper="-0.785398163397" velocity="10.0" effort="200.0"/>
-        <origin xyz="0.0 0.175 0.0" rpy="0 0 0"/>
-        <axis xyz="0 0 1"/>
-        <joint_properties damping="6.0" friction="6.0"/>
+        <limit lower="-0.785398163397 " upper="0.785398163397" velocity="10.0" effort="200.0"/>
+        <origin xyz="0.0 0.175 0.0" rpy="0 0 0"/>
+        <axis xyz="0 0 1"/>
+        <joint_properties damping="2.0" friction="2.0"/>
     </joint>
     <!-- LINK 3 -->
@@ -90,8 +90,8 @@
         <parent link="link_3"/>
         <child link="link_4"/>
-        <limit lower="0.785398163397 " upper="-0.785398163397" velocity="10.0" effort="200.0"/>
-        <origin xyz="0.0 0.175 0.0" rpy="0 0 0"/>
-        <axis xyz="0 0 1"/>
-        <joint_properties damping="6.0" friction="6.0"/>
+        <limit lower="-0.785398163397 " upper="0.785398163397" velocity="10.0" effort="200.0"/>
+        <origin xyz="0.0 0.175 0.0" rpy="0 0 0"/>
+        <axis xyz="0 0 1"/>
+        <joint_properties damping="2.0" friction="2.0"/>
     </joint>
     <!-- LINK 4 -->
@@ -117,8 +117,8 @@
         <parent link="link_4"/>
         <child link="link_5"/>
-        <limit lower="0.785398163397 " upper="-0.785398163397" velocity="10.0" effort="200.0"/>
-        <origin xyz="0.0 0.175 0.0" rpy="0 0 0"/>
-        <axis xyz="0 0 1"/>
-        <joint_properties damping="6.0" friction="6.0"/>
+        <limit lower="-0.785398163397 " upper="0.785398163397" velocity="10.0" effort="200.0"/>
+        <origin xyz="0.0 0.175 0.0" rpy="0 0 0"/>
+        <axis xyz="0 0 1"/>
+        <joint_properties damping="2.0" friction="2.0"/>
     </joint>
     <!-- LINK 5-->
@@ -144,8 +144,8 @@
         <parent link="link_5"/>
         <child link="link_6"/>
-        <limit lower="0.785398163397 " upper="-0.785398163397" velocity="10.0" effort="200.0"/>
-        <origin xyz="0.0 0.175 0.0" rpy="0 0 0"/>
-        <axis xyz="0 0 1"/>
-        <joint_properties damping="6.0" friction="6.0"/>
+        <limit lower="-0.785398163397 " upper="0.785398163397" velocity="10.0" effort="200.0"/>
+        <origin xyz="0.0 0.175 0.0" rpy="0 0 0"/>
+        <axis xyz="0 0 1"/>
+        <joint_properties damping="2.0" friction="2.0"/>
     </joint>
     <!--  LINK 6-->
@@ -172,8 +172,8 @@
         <parent link="link_6"/>
         <child link="link_7"/>
-        <limit lower="0.785398163397 " upper="-0.785398163397" velocity="10.0" effort="200.0"/>
-        <origin xyz="0.0 0.175 0.0" rpy="0 0 0"/>
-        <axis xyz="0 0 1"/>
-        <joint_properties damping="6.0" friction="6.0"/>
+        <limit lower="-0.785398163397 " upper="0.785398163397" velocity="10.0" effort="200.0"/>
+        <origin xyz="0.0 0.175 0.0" rpy="0 0 0"/>
+        <axis xyz="0 0 1"/>
+        <joint_properties damping="2.0" friction="2.0"/>
     </joint>
     <!--  LINK 7-->
@@ -200,8 +200,8 @@
         <parent link="link_7"/>
         <child link="link_8"/>
-        <limit lower="0.785398163397 " upper="-0.785398163397" velocity="10.0" effort="200.0"/>
-        <origin xyz="0.0 0.175 0.0" rpy="0 0 0"/>
-        <axis xyz="0 0 1"/>
-        <joint_properties damping="6.0" friction="6.0"/>
+        <limit lower="-0.785398163397 " upper="0.785398163397" velocity="10.0" effort="200.0"/>
+        <origin xyz="0.0 0.175 0.0" rpy="0 0 0"/>
+        <axis xyz="0 0 1"/>
+        <joint_properties damping="2.0" friction="2.0"/>
     </joint>
     <!--  LINK 8-->
@@ -228,8 +228,8 @@
         <parent link="link_8"/>
         <child link="link_9"/>
-        <limit lower="0.785398163397 " upper="-0.785398163397" velocity="10.0" effort="200.0"/>
-        <origin xyz="0.0 0.175 0.0" rpy="0 0 0"/>
-        <axis xyz="0 0 1"/>
-        <joint_properties damping="6.0" friction="6.0"/>
+        <limit lower="-0.785398163397 " upper="0.785398163397" velocity="10.0" effort="200.0"/>
+        <origin xyz="0.0 0.175 0.0" rpy="0 0 0"/>
+        <axis xyz="0 0 1"/>
+        <joint_properties damping="2.0" friction="2.0"/>
     </joint>
     <!--  LINK 9-->
@@ -256,8 +256,8 @@
         <parent link="link_9"/>
         <child link="link_10"/>
-        <limit lower="-0.785398163397 " upper="0.785398163397" velocity="10" effort="200.0"/>
-        <origin xyz="0.0 0.175 0.0" rpy="0 0 0"/>
-        <axis xyz="0 0 1"/>
-        <joint_properties damping="6.0" friction="6.0"/>
+        <limit lower="-0.785398163397 " upper="0.785398163397" velocity="10.0" effort="200.0"/>
+        <origin xyz="0.0 0.175 0.0" rpy="0 0 0"/>
+        <axis xyz="0 0 1"/>
+        <joint_properties damping="2.0" friction="2.0"/>
     </joint>
     <!--  LINK 10-->

Commit message: new

File: description/ros2_control.xacro (robot description, xacro)
@@ -47,5 +47,5 @@
     </gazebo>
     <gazebo reference="link_10">
-        <material>Gazebo/Black</material>
+        <material>Gazebo/Blue</material>
         <mu1>0.1</mu1>
         <mu2>1</mu2>

File: description/snake_robot_core.xacro (robot description, xacro)
@@ -36,5 +36,5 @@
         <limit lower="-0.785398163397 " upper="0.785398163397" velocity="10.0" effort="200.0"/>
         <origin xyz="0.0 0.175 0.0" rpy="0 0 0"/>
-        <axis xyz="0 0 1"/>
+        <axis xyz=" 0 0 1 "/>
         <joint_properties damping="8.0" friction="2.0"/>
     </joint>
@@ -64,5 +64,5 @@
         <limit lower="-0.785398163397 " upper="0.785398163397" velocity="10.0" effort="200.0"/>
         <origin xyz="0.0 0.175 0.0" rpy="0 0 0"/>
-        <axis xyz="0 0 1"/>
+        <axis xyz=" 0 0 1 "/>
         <joint_properties damping="8.0" friction="2.0"/>
     </joint>
@@ -92,5 +92,5 @@
         <limit lower="-0.785398163397 " upper="0.785398163397" velocity="10.0" effort="200.0"/>
         <origin xyz="0.0 0.175 0.0" rpy="0 0 0"/>
-        <axis xyz="0 0 1"/>
+        <axis xyz=" 0 0 1 "/>
         <joint_properties damping="8.0" friction="2.0"/>
     </joint>
@@ -119,5 +119,5 @@
         <limit lower="-0.785398163397 " upper="0.785398163397" velocity="10.0" effort="200.0"/>
         <origin xyz="0.0 0.175 0.0" rpy="0 0 0"/>
-        <axis xyz="0 0 1"/>
+        <axis xyz=" 0 0 1 "/>
         <joint_properties damping="8.0" friction="2.0"/>
     </joint>
@@ -146,5 +146,5 @@
         <limit lower="-0.785398163397 " upper="0.785398163397" velocity="10.0" effort="200.0"/>
         <origin xyz="0.0 0.175 0.0" rpy="0 0 0"/>
-        <axis xyz="0 0 1"/>
+        <axis xyz=" 0 0 1 "/>
         <joint_properties damping="8.0" friction="2.0"/>
     </joint>
@@ -174,5 +174,5 @@
         <limit lower="-0.785398163397 " upper="0.785398163397" velocity="10.0" effort="200.0"/>
         <origin xyz="0.0 0.175 0.0" rpy="0 0 0"/>
-        <axis xyz="0 0 1"/>
+        <axis xyz=" 0 0 1 "/>
         <joint_properties damping="8.0" friction="2.0"/>
     </joint>
@@ -202,5 +202,5 @@
         <limit lower="-0.785398163397 " upper="0.785398163397" velocity="10.0" effort="200.0"/>
         <origin xyz="0.0 0.175 0.0" rpy="0 0 0"/>
-        <axis xyz="0 0 1"/>
+        <axis xyz=" 0 0 1 "/>
         <joint_properties damping="8.0" friction="2.0"/>
     </joint>
@@ -230,5 +230,5 @@
         <limit lower="-0.785398163397 " upper="0.785398163397" velocity="10.0" effort="200.0"/>
         <origin xyz="0.0 0.175 0.0" rpy="0 0 0"/>
-        <axis xyz="0 0 1"/>
+        <axis xyz=" 0 0 1 "/>
         <joint_properties damping="8.0" friction="2.0"/>
     </joint>
@@ -258,5 +258,5 @@
         <limit lower="-0.785398163397 " upper="0.785398163397" velocity="10.0" effort="200.0"/>
         <origin xyz="0.0 0.175 0.0" rpy="0 0 0"/>
-        <axis xyz="0 0 1"/>
+        <axis xyz=" 0 0 1 "/>
         <joint_properties damping="8.0" friction="2.0"/>
     </joint>
@@ -264,5 +264,5 @@
     <link name="link_10">
         <visual>
-            <material name="black"/>
+            <material name="blue"/>
             <origin xyz="0.0 0.07 0.03" rpy="0.0 0.0 0.0"/>
             <geometry>
