Commit message: new

File: description/ros2_control.xacro (robot description, xacro)
@@ -3,51 +3,51 @@
      <gazebo reference="link_1">
         <material>Gazebo/Orange</material>
-        <mu1>0.1</mu1>
-        <mu2>1</mu2>
+        <mu1>0.7</mu1>
+        <mu2>0.9</mu2>
     </gazebo>
     <gazebo reference="link_2">
         <material>Gazebo/Black</material>
-        <mu1>0.1</mu1>
-        <mu2>1</mu2>
+        <mu1>0.7</mu1>
+        <mu2>0.9</mu2>
     </gazebo>
     <gazebo reference="link_3">
         <material>Gazebo/Orange</material>
-        <mu1>0.1</mu1>
-        <mu2>1</mu2>
+        <mu1>0.7</mu1>
+        <mu2>0.9</mu2>
     </gazebo>
     <gazebo reference="link_4">
         <material>Gazebo/Black</material>
-        <mu1>0.1</mu1>
-        <mu2>1</mu2>
+        <mu1>0.7</mu1>
+        <mu2>0.9</mu2>
     </gazebo>
     <gazebo reference="link_5">
         <material>Gazebo/Orange</material>
-        <mu1>0.1</mu1>
-        <mu2>1</mu2>
+        <mu1>0.7</mu1>
+        <mu2>0.9</mu2>
     </gazebo>
     <gazebo reference="link_6">
         <material>Gazebo/Black</material>
-        <mu1>0.1</mu1>
-        <mu2>1</mu2>
+        <mu1>0.7</mu1>
+        <mu2>0.9</mu2>
     </gazebo>
     <gazebo reference="link_7">
         <material>Gazebo/Orange</material>
-        <mu1>0.1</mu1>
-        <mu2>1</mu2>
+        <mu1>0.7</mu1>
+        <mu2>0.9</mu2>
     </gazebo>
     <gazebo reference="link_8">
         <material>Gazebo/Black</material>
-        <mu1>0.1</mu1>
-        <mu2>1</mu2>
+        <mu1>0.7</mu1>
+        <mu2>0.9</mu2>
     </gazebo>
     <gazebo reference="link_9">
         <material>Gazebo/Orange</material>
-        <mu1>0.1</mu1>
-        <mu2>1</mu2>
+        <mu1>0.7</mu1>
+        <mu2>0.9</mu2>
     </gazebo>
     <gazebo reference="link_10">
         <material>Gazebo/Blue</material>
-        <mu1>0.1</mu1>
-        <mu2>1</mu2>
+        <mu1>0.7</mu1>
+        <mu2>0.9</mu2>
     </gazebo>
     <ros2_control name="GazeboSystem" type="system">

File: description/snake_robot_core.xacro (robot description, xacro)
@@ -27,5 +27,5 @@
         </collision>
         <xacro:inertial_box mass="1" x="0.06" y="0.14" z="0.06">
-            <origin xyz="0.03 0.07 0.03" rpy="0.0 0.0 0.0"/>
+            <origin xyz="0.0 0.07 0.03" rpy="0.0 0.0 0.0"/>
         </xacro:inertial_box>
     </link>
@@ -55,5 +55,5 @@
         </collision>
         <xacro:inertial_box mass="1" x="0.06" y="0.14" z="0.06">
-            <origin xyz="0.03 0.07 0.03" rpy="0.0 0.0 0.0"/>
+            <origin xyz="0.0 0.07 0.03" rpy="0.0 0.0 0.0"/>
         </xacro:inertial_box>
     </link>
@@ -62,5 +62,6 @@
         <parent link="link_2"/>
         <child link="link_3"/>
-        <limit lower="-0.785398163397 " upper="0.785398163397" velocity="10.0" effort="200.0"/>
+        <limit lower="-0.785398163397 " upper="0.785398163397"
+        velocity="10.0" effort="200.0"/>
         <origin xyz="0.0 0.175 0.0" rpy="0 0 0"/>
         <axis xyz=" 0 0 1 "/>
@@ -83,5 +84,5 @@
         </collision>
         <xacro:inertial_box mass="1" x="0.06" y="0.14" z="0.06">
-            <origin xyz="0.03 0.07 0.03" rpy="0.0 0.0 0.0"/>
+            <origin xyz="0.0 0.07 0.03" rpy="0.0 0.0 0.0"/>
         </xacro:inertial_box>
     </link>
@@ -111,5 +112,5 @@
         </collision>
         <xacro:inertial_box mass="1" x="0.06" y="0.14" z="0.06">
-            <origin xyz="0.03 0.07 0.03" rpy="0.0 0.0 0.0"/>
+            <origin xyz="0.0 0.07 0.03" rpy="0.0 0.0 0.0"/>
         </xacro:inertial_box>
     </link>
@@ -138,5 +139,5 @@
         </collision>
         <xacro:inertial_box mass="1" x="0.06" y="0.14" z="0.06">
-            <origin xyz="0.03 0.07 0.03" rpy="0.0 0.0 0.0"/>
+            <origin xyz="0.0 0.07 0.03" rpy="0.0 0.0 0.0"/>
         </xacro:inertial_box>
     </link>
@@ -165,5 +166,5 @@
         </collision>
         <xacro:inertial_box mass="1" x="0.06" y="0.14" z="0.06">
-            <origin xyz="0.03 0.07 0.03" rpy="0.0 0.0 0.0"/>
+            <origin xyz="0.0 0.07 0.03" rpy="0.0 0.0 0.0"/>
         </xacro:inertial_box>
     </link>
@@ -193,5 +194,5 @@
         </collision>
         <xacro:inertial_box mass="1" x="0.06" y="0.14" z="0.06">
-            <origin xyz="0.03 0.07 0.03" rpy="0.0 0.0 0.0"/>
+            <origin xyz="0.0 0.07 0.03" rpy="0.0 0.0 0.0"/>
         </xacro:inertial_box>
     </link>
@@ -221,5 +222,5 @@
         </collision>
         <xacro:inertial_box mass="1" x="0.06" y="0.14" z="0.06">
-            <origin xyz="0.03 0.07 0.03" rpy="0.0 0.0 0.0"/>
+            <origin xyz="0.0 0.07 0.03" rpy="0.0 0.0 0.0"/>
         </xacro:inertial_box>
     </link>
@@ -249,5 +250,5 @@
         </collision>
         <xacro:inertial_box mass="1" x="0.06" y="0.14" z="0.06">
-            <origin xyz="0.03 0.07 0.03" rpy="0.0 0.0 0.0"/>
+            <origin xyz="0.0 0.07 0.03" rpy="0.0 0.0 0.0"/>
         </xacro:inertial_box>
     </link>
@@ -261,5 +262,5 @@
         <joint_properties damping="8.0" friction="2.0"/>
     </joint>
-    <!--  LINK 10-->
+    <!--  LINK 10 or Head link-->
     <link name="link_10">
         <visual>
@@ -277,5 +278,5 @@
         </collision>
         <xacro:inertial_box mass="1" x="0.06" y="0.14" z="0.06">
-            <origin xyz="0.03 0.07 0.03" rpy="0.0 0.0 0.0"/>
+            <origin xyz="0.0 0.07 0.03" rpy="0.0 0.0 0.0"/>
         </xacro:inertial_box>
     </link>
